File: EasyBMS.sch (EAGLE design)
At the start: 154 parts, among them Q1 C8547, Q10 C8547, Q11 C8547, Q12 C8547, Q13 C8547, Q2 C8547, Q4 C8547, Q5 C8547, Q6 C8547, Q7 C8547, Q8 C8547, Q9 C8547

Commit message: add vias, fix with battery measurement
Parts:
- added H1, H2, H3, H4: MOUNT-PAD-ROUND3.2, holes:MOUNT-PAD-ROUND3.2
Connections:
- removed net BAT+: R15.2, R59.2
- net GND: now also H1.MOUNT, H2.MOUNT, H3.MOUNT, H4.MOUNT
- net P13: now also R15.2, R59.2
Changed lines of the file:
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@@
 <part name="R95" library="rcl" library_urn="urn:adsk.eagle:library:334" deviceset="R-EU_" device="R0402" package3d_urn="urn:adsk.eagle:package:23547/1" value="470R"/>
 <part name="R96" library="rcl" library_urn="urn:adsk.eagle:library:334" deviceset="R-EU_" device="R0402" package3d_urn="urn:adsk.eagle:package:23547/1" value="100R"/>
+<part name="H1" library="holes" library_urn="urn:adsk.eagle:library:237" deviceset="MOUNT-PAD-ROUND" device="3.2" package3d_urn="urn:adsk.eagle:package:14282/1" value="MOUNT-PAD-ROUND3.2"/>
+<part name="H2" library="holes" library_urn="urn:adsk.eagle:library:237" deviceset="MOUNT-PAD-ROUND" device="3.2" package3d_urn="urn:adsk.eagle:package:14282/1" value="MOUNT-PAD-ROUND3.2"/>
+<part name="H3" library="holes" library_urn="urn:adsk.eagle:library:237" deviceset="MOUNT-PAD-ROUND" device="3.2" package3d_urn="urn:adsk.eagle:package:14282/1" value="MOUNT-PAD-ROUND3.2"/>
+<part name="H4" library="holes" library_urn="urn:adsk.eagle:library:237" deviceset="MOUNT-PAD-ROUND" device="3.2" package3d_urn="urn:adsk.eagle:package:14282/1" value="MOUNT-PAD-ROUND3.2"/>
+<part name="GND1" library="supply1" library_urn="urn:adsk.eagle:library:371" deviceset="GND" device=""/>
+<part name="GND2" library="supply1" library_urn="urn:adsk.eagle:library:371" deviceset="GND" device=""/>
+<part name="GND3" library="supply1" library_urn="urn:adsk.eagle:library:371" deviceset="GND" device=""/>
+<part name="GND4" library="supply1" library_urn="urn:adsk.eagle:library:371" deviceset="GND" device=""/>
+<part name="GND5" library="supply1" library_urn="urn:adsk.eagle:library:371" deviceset="GND" device=""/>
+<part name="GND6" library="supply1" library_urn="urn:adsk.eagle:library:371" deviceset="GND" device=""/>
+<part name="GND7" library="supply1" library_urn="urn:adsk.eagle:library:371" deviceset="GND" device=""/>
+<part name="GND8" library="supply1" library_urn="urn:adsk.eagle:library:371" deviceset="GND" device=""/>
+<part name="GND9" library="supply1" library_urn="urn:adsk.eagle:library:371" deviceset="GND" device=""/>
 </parts>
 <sheets>
@@
 <attribute name="VALUE" x="280.67" y="790.702" size="1.778" layer="96" rot="R180"/>
 </instance>
+<instance part="H1" gate="G$1" x="868.68" y="314.96" smashed="yes">
+<attribute name="NAME" x="871.474" y="315.5442" size="1.778" layer="95"/>
+<attribute name="VALUE" x="871.474" y="312.4962" size="1.778" layer="96"/>
+</instance>
+<instance part="H2" gate="G$1" x="904.24" y="314.96" smashed="yes">
+<attribute name="NAME" x="907.034" y="315.5442" size="1.778" layer="95"/>
+<attribute name="VALUE" x="907.034" y="312.4962" size="1.778" layer="96"/>
+</instance>
+<instance part="H3" gate="G$1" x="904.24" y="302.26" smashed="yes">
+<attribute name="NAME" x="907.034" y="302.8442" size="1.778" layer="95"/>
+<attribute name="VALUE" x="907.034" y="299.7962" size="1.778" layer="96"/>
+</instance>
+<instance part="H4" gate="G$1" x="868.68" y="302.26" smashed="yes">
+<attribute name="NAME" x="871.474" y="302.8442" size="1.778" layer="95"/>
+<attribute name="VALUE" x="871.474" y="299.7962" size="1.778" layer="96"/>
+</instance>
+<instance part="GND1" gate="1" x="1176.02" y="175.26" smashed="yes">
+<attribute name="VALUE" x="1173.48" y="172.72" size="1.778" layer="96"/>
+</instance>
+<instance part="GND2" gate="1" x="1216.66" y="175.26" smashed="yes">
+<attribute name="VALUE" x="1214.12" y="172.72" size="1.778" layer="96"/>
+</instance>
+<instance part="GND3" gate="1" x="975.36" y="71.12" smashed="yes">
+<attribute name="VALUE" x="972.82" y="68.58" size="1.778" layer="96"/>
+</instance>
+<instance part="GND4" gate="1" x="868.68" y="426.72" smashed="yes">
+<attribute name="VALUE" x="866.14" y="424.18" size="1.778" layer="96"/>
+</instance>
+<instance part="GND5" gate="1" x="767.08" y="271.78" smashed="yes">
+<attribute name="VALUE" x="764.54" y="269.24" size="1.778" layer="96"/>
+</instance>
+<instance part="GND6" gate="1" x="457.2" y="63.5" smashed="yes">
+<attribute name="VALUE" x="454.66" y="60.96" size="1.778" layer="96"/>
+</instance>
+<instance part="GND7" gate="1" x="1234.44" y="220.98" smashed="yes">
+<attribute name="VALUE" x="1231.9" y="218.44" size="1.778" layer="96"/>
+</instance>
+<instance part="GND8" gate="1" x="863.6" y="289.56" smashed="yes">
+<attribute name="VALUE" x="861.06" y="287.02" size="1.778" layer="96"/>
+</instance>
+<instance part="GND9" gate="1" x="899.16" y="289.56" smashed="yes">
+<attribute name="VALUE" x="896.62" y="287.02" size="1.778" layer="96"/>
+</instance>
 </instances>
 <busses>
 </busses>
 <nets>
-<net name="BAT+" class="0">
-<segment>
-<pinref part="R15" gate="G$1" pin="2"/>
-<wire x1="1216.66" y1="203.2" x2="1216.66" y2="205.74" width="0.1524" layer="91"/>
-<label x="1216.66" y="205.74" size="1.778" layer="95"/>
-</segment>
-<segment>
-<pinref part="R59" gate="G$1" pin="2"/>
-<wire x1="1176.02" y1="203.2" x2="1176.02" y2="205.74" width="0.1524" layer="91"/>
-<label x="1178.56" y="205.74" size="1.778" layer="95"/>
-</segment>
-</net>
 <net name="5VDC" class="0">
 <segment>
@@
 <wire x1="1211.58" y1="231.14" x2="1216.66" y2="231.14" width="0.1524" layer="91"/>
 <wire x1="1211.58" y1="231.14" x2="1211.58" y2="223.52" width="0.1524" layer="91"/>
-<wire x1="1211.58" y1="223.52" x2="1257.3" y2="223.52" width="0.1524" layer="91"/>
+<wire x1="1211.58" y1="223.52" x2="1234.44" y2="223.52" width="0.1524" layer="91"/>
+<wire x1="1234.44" y1="223.52" x2="1257.3" y2="223.52" width="0.1524" layer="91"/>
 <wire x1="1257.3" y1="223.52" x2="1257.3" y2="231.14" width="0.1524" layer="91"/>
 <junction x="1257.3" y="231.14"/>
@@
 <wire x1="975.36" y1="106.68" x2="975.36" y2="73.66" width="0.1524" layer="91"/>
 <junction x="975.36" y="73.66"/>
+<pinref part="GND3" gate="1" pin="GND"/>
+<pinref part="GND7" gate="1" pin="GND"/>
+<junction x="1234.44" y="223.52"/>
 </segment>
 <segment>
@@
 <wire x1="1216.66" y1="180.34" x2="1216.66" y2="177.8" width="0.1524" layer="91"/>
 <label x="1216.66" y="177.8" size="1.778" layer="95"/>
+<pinref part="GND2" gate="1" pin="GND"/>
 </segment>
 <segment>
@@
 <wire x1="756.92" y1="289.56" x2="756.92" y2="274.32" width="0.1524" layer="91"/>
 <pinref part="R58" gate="G$1" pin="1"/>
-<wire x1="756.92" y1="274.32" x2="774.7" y2="274.32" width="0.1524" layer="91"/>
+<wire x1="756.92" y1="274.32" x2="767.08" y2="274.32" width="0.1524" layer="91"/>
+<wire x1="767.08" y1="274.32" x2="774.7" y2="274.32" width="0.1524" layer="91"/>
 <wire x1="774.7" y1="274.32" x2="774.7" y2="289.56" width="0.1524" layer="91"/>
 <label x="764.54" y="274.32" size="1.778" layer="95"/>
+<pinref part="GND5" gate="1" pin="GND"/>
+<junction x="767.08" y="274.32"/>
 </segment>
 <segment>
@@
 <wire x1="1176.02" y1="180.34" x2="1176.02" y2="177.8" width="0.1524" layer="91"/>
 <label x="1170.94" y="175.26" size="1.778" layer="95"/>
+<pinref part="GND1" gate="1" pin="GND"/>
 </segment>
 <segment>
@@
 <wire x1="868.68" y1="436.88" x2="868.68" y2="429.26" width="0.1524" layer="91"/>
 <label x="861.06" y="429.26" size="1.778" layer="95"/>
+<pinref part="GND4" gate="1" pin="GND"/>
 </segment>
 <segment>
@@
 <wire x1="431.8" y1="68.58" x2="431.8" y2="66.04" width="0.1524" layer="91"/>
 <junction x="431.8" y="66.04"/>
+<pinref part="GND6" gate="1" pin="GND"/>
+</segment>
+<segment>
+<pinref part="GND8" gate="1" pin="GND"/>
+<pinref part="H1" gate="G$1" pin="MOUNT"/>
+<wire x1="863.6" y1="292.1" x2="863.6" y2="302.26" width="0.1524" layer="91"/>
+<wire x1="863.6" y1="302.26" x2="863.6" y2="314.96" width="0.1524" layer="91"/>
+<wire x1="863.6" y1="314.96" x2="866.14" y2="314.96" width="0.1524" layer="91"/>
+<pinref part="H4" gate="G$1" pin="MOUNT"/>
+<wire x1="863.6" y1="302.26" x2="866.14" y2="302.26" width="0.1524" layer="91"/>
+<junction x="863.6" y="302.26"/>
+</segment>
+<segment>
+<pinref part="GND9" gate="1" pin="GND"/>
+<pinref part="H2" gate="G$1" pin="MOUNT"/>
+<wire x1="899.16" y1="292.1" x2="899.16" y2="302.26" width="0.1524" layer="91"/>
+<wire x1="899.16" y1="302.26" x2="899.16" y2="314.96" width="0.1524" layer="91"/>
+<wire x1="899.16" y1="314.96" x2="901.7" y2="314.96" width="0.1524" layer="91"/>
+<pinref part="H3" gate="G$1" pin="MOUNT"/>
+<wire x1="901.7" y1="302.26" x2="899.16" y2="302.26" width="0.1524" layer="91"/>
+<junction x="899.16" y="302.26"/>
 </segment>
 </net>
@@
 <label x="223.52" y="787.4" size="1.778" layer="95"/>
 </segment>
-</net>
+<segment>
+<pinref part="R59" gate="G$1" pin="2"/>
+<wire x1="1176.02" y1="203.2" x2="1176.02" y2="205.74" width="0.1524" layer="91"/>
+<label x="1178.56" y="205.74" size="1.778" layer="95"/>
+</segment>
+<segment>
+<pinref part="R15" gate="G$1" pin="2"/>
+<wire x1="1216.66" y1="203.2" x2="1216.66" y2="205.74" width="0.1524" layer="91"/>
+<label x="1216.66" y="205.74" size="1.778" layer="95"/>
+</segment>
+</net>

Commit message: added jumper for connecting any cell to V+ reworked jumper on C pins for easier handling
Parts:
- added JP13: (no value), pinhead:PINHD-2X5
- added JP14: (no value), pinhead:PINHD-2X6
- JP11: value UpperADC -> (none); device pinhead:PINHD-2X6 -> pinhead:PINHD-2X5
- JP12: value LowerADC -> (none); device pinhead:PINHD-2X6 -> pinhead:PINHD-2X5
Connections:
- removed net N$106: JP12.10, JP12.12, JP12.2, JP12.4, JP12.6, JP12.8
- removed net N$121: JP11.10, JP11.12, JP11.2, JP11.4, JP11.6, JP11.8
- net C1: now also JP12.9; no longer JP12.11
- net C10: now also JP11.3; no longer JP11.5
- net C11: now also JP11.1; no longer JP11.3
- net C12: now also JP11.10, JP11.2, JP11.4, JP11.6, JP11.8; no longer JP11.1
- net C2: now also JP12.7; no longer JP12.9
- net C3: now also JP12.5; no longer JP12.7
- net C4: now also JP12.3; no longer JP12.5
- net C5: now also JP12.1; no longer JP12.3
- net C6: now also JP12.10, JP12.2, JP12.4, JP12.6, JP12.8; no longer JP12.1
- net C7: now also JP11.9; no longer JP11.11
- net C8: now also JP11.7; no longer JP11.9
- net C9: now also JP11.5; no longer JP11.7
- net P10: now also JP13.6
- net P11: now also JP13.4
- net P12: now also JP13.2
- net P13: now also JP13.1, JP13.3, JP13.5, JP13.7, JP13.9, JP14.1
- net P2: now also JP14.12
- net P3: now also JP14.10
- net P4: now also JP14.8
- net P5: now also JP14.6
- net P6: now also JP14.4
- net P7: now also JP14.11, JP14.2, JP14.3, JP14.5, JP14.7, JP14.9
- net P8: now also JP13.10
- net P9: now also JP13.8
Other:
- moved on the sheet: C10, C11, C12, C13, C14, C15, C17, C20, C4, C5, C7, C8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
