File: CurrentSensorAC712-30.brd (EAGLE design)
At the start: 48 x 24 mm, 9 parts, among them IC1 ACS758LCB-050B-PFF-T

Commit message: new footprint for current sensor added
Parts:
- added C2: 10nF, rcl:C0805
- added R2: 10k, rcl:R0805
- moved JP2 1.27 mm to (10.2, 20.3)
- moved JP3 1.27 mm to (10.2, 3.81)
- moved LED1 0.76 mm to (6.86, 21.8), turned to 0 degrees
Connections:
- new net N$1: IC1.3, R2.1
- net GND: now also C2.1
- net N$6: now also C2.2, R2.2; no longer IC1.3
Routing:
- net GND: track 3.98 -> 8.71 mm
- net N$1: track 0.00 -> 2.59 mm
- net N$5: track 3.12 -> 2.49 mm
