File: GPIO_Adapter.sch (EAGLE design)
At the start: 1 part

Commit message: GPIO got terminal blocks
Parts:
- added JP10, JP11, JP12, JP13, JP14, JP15, JP3, JP4, JP5, JP6, JP7, JP8, JP9: (no value), pinhead:PINHD-1X3
- added R1, R11, R13, R15, R17, R19, R21, R23, R25, R27, R29, R5, R7, R9: 7k5, rcl:R-EU_R0805
- added R10, R12, R14, R16, R18, R2, R20, R22, R24, R26, R28, R30, R6, R8: 2k7, rcl:R-EU_R0805
- added U$1: DC-DC-STEP-DOWN-LM2596HVS, diy-modules:DC-DC-STEP-DOWN-LM2596HVS
- added X1: RASPI_BOARD_B+#_F, raspberrypi_bastelstube_v13:RASPI_BOARD_B+#_F
- added X2: MKDSN1,5/8-5,08, con-phoenix-508:MKDSN1,5/8-5,08
- added X3: MKDSN1,5/10-5,08, con-phoenix-508:MKDSN1,5/10-5,08
- JP1: device pinhead:PINHD-2X20 -> pinhead:PINHD-1X3
Connections:
- removed net N$19: JP1.37
- removed net N$20 (its old number): JP1.39
- new net 3,3V: X1.3V3A, X1.3V3B
- new net 5VDC: U$1.OUT+, X1.5V0A, X1.5V0B
- new net GND: R10.2, R12.2, R14.2, R16.2, R18.2, R2.2, R20.2, R22.2, R24.2, R26.2, R28.2, R30.2, R6.2, R8.2, U$1.IN-, U$1.OUT-, X1.GND_A, X1.GND_B, X1.GND_C, X1.GND_D, X1.GND_E, X1.GND_F, X1.GND_G, X1.GND_H, X3-2.KL
- new net N$40: JP9.3, R17.2, R18.1
- new net N$41: JP9.2
- new net N$42: JP10.1, R19.1
- new net N$43: JP10.3, R19.2, R20.1
- new net N$44: JP10.2
- new net N$45: JP11.1, R21.1
- new net N$46: JP11.3, R21.2, R22.1
- new net N$47: JP11.2
- new net N$48: JP12.1, R23.1
- new net N$49: JP12.3, R23.2, R24.1
- new net N$50: JP12.2
- new net N$51: JP13.1, R25.1
- new net N$52: JP13.3, R25.2, R26.1
- new net N$53: JP13.2
- new net N$54: JP14.1, R27.1
- new net N$55: JP14.3, R27.2, R28.1
- new net N$56: JP14.2
- new net N$57: JP15.1, R29.1
- new net N$58: JP15.3, R29.2, R30.1
- new net N$59: JP15.2
- new net VIN: U$1.IN+, X3-1.KL
- net N$1: now also X2-1.KL; no longer JP1.1
- net N$10: now also JP1.3, R1.2, R2.1; no longer JP1.19
- net N$11: now also X3-3.KL; no longer JP1.21
- net N$12: now also X3-4.KL; no longer JP1.23
- net N$13: now also X3-5.KL; no longer JP1.25
- net N$14: now also X3-6.KL; no longer JP1.27
- net N$15: now also X3-7.KL; no longer JP1.29
- net N$16: now also X3-8.KL; no longer JP1.31
- net N$17: now also X3-9.KL; no longer JP1.33
- net N$18: now also X3-10.KL; no longer JP1.35
- net N$2: now also X2-2.KL; no longer JP1.3
- net N$21: now also JP3.1, R5.1; no longer JP1.40
- net N$22: now also JP3.3, R5.2, R6.1; no longer JP1.38
- net N$23: now also JP3.2; no longer JP1.36
- net N$24: now also JP4.1, R7.1; no longer JP1.34
- net N$25: now also JP4.3, R7.2, R8.1; no longer JP1.32
- net N$26: now also JP4.2; no longer JP1.30
- net N$27: now also JP5.1, R9.1; no longer JP1.28
- net N$28: now also JP5.3, R10.1, R9.2; no longer JP1.26
- net N$29: now also JP5.2; no longer JP1.24
- net N$3: now also X2-3.KL; no longer JP1.5
- net N$30: now also JP6.1, R11.1; no longer JP1.22
- net N$31: now also JP6.3, R11.2, R12.1; no longer JP1.20
- net N$32: now also JP6.2; no longer JP1.18
- net N$33: now also JP7.1, R13.1; no longer JP1.16
- net N$34: now also JP7.3, R13.2, R14.1; no longer JP1.14
- net N$35: now also JP7.2; no longer JP1.12
- net N$36: now also JP8.1, R15.1; no longer JP1.10
- net N$37: now also JP8.3, R15.2, R16.1; no longer JP1.8
- net N$38: now also JP8.2; no longer JP1.6
- net N$39: now also JP9.1, R17.1; no longer JP1.4
- net N$4: now also X2-4.KL; no longer JP1.7
- net N$5: now also X2-5.KL; no longer JP1.9
- net N$6: now also X2-6.KL; no longer JP1.11
- net N$7: now also X2-7.KL; no longer JP1.13
- net N$8: now also X2-8.KL; no longer JP1.15
- net N$9: now also JP1.1, R1.1; no longer JP1.17

Commit message: GPIO board ready for manufactoring
Connections:
- removed net 3,3V: X1.3V3A, X1.3V3B
- removed net N$1: X2-1.KL
- removed net N$10: JP1.3, R1.2, R2.1
- removed net N$11: X3-3.KL
- removed net N$12: X3-4.KL
- removed net N$13: X3-5.KL
- removed net N$14: X3-6.KL
- removed net N$15: X3-7.KL
- removed net N$16: X3-8.KL
- removed net N$17: X3-9.KL
- removed net N$18: X3-10.KL
- removed net N$2: X2-2.KL
- removed net N$20: JP1.2
- removed net N$22: JP3.3, R5.2, R6.1
- removed net N$23: JP3.2
- removed net N$25: JP4.3, R7.2, R8.1
- removed net N$26: JP4.2
- removed net N$28: JP5.3, R10.1, R9.2
- removed net N$29: JP5.2
- removed net N$3: X2-3.KL
- removed net N$31: JP6.3, R11.2, R12.1
- removed net N$32: JP6.2
- removed net N$34: JP7.3, R13.2, R14.1
- removed net N$35: JP7.2
- removed net N$37: JP8.3, R15.2, R16.1
- removed net N$38: JP8.2
- removed net N$4: X2-4.KL
- removed net N$40: JP9.3, R17.2, R18.1
- removed net N$41: JP9.2
- removed net N$43: JP10.3, R19.2, R20.1
- removed net N$44: JP10.2
- removed net N$46: JP11.3, R21.2, R22.1
- removed net N$47: JP11.2
- removed net N$49: JP12.3, R23.2, R24.1
- removed net N$5: X2-5.KL
- removed net N$50: JP12.2
- removed net N$52: JP13.3, R25.2, R26.1
- removed net N$53: JP13.2
- removed net N$55: JP14.3, R27.2, R28.1
- removed net N$56: JP14.2
- removed net N$58: JP15.3, R29.2, R30.1
- removed net N$59: JP15.2
- removed net N$6: X2-6.KL
- removed net N$7: X2-7.KL
- removed net N$8: X2-8.KL
- new net 3.3V: X1.3V3A, X1.3V3B, X2-2.KL
- new net GPIO12: JP5.3, R10.1, R9.2, X1.GPIO12
- new net GPIO12EXT: JP5.2, X3-6.KL
- new net GPIO13: JP6.3, R11.2, R12.1, X1.GPIO13
- new net GPIO13EXT: JP6.2, X3-7.KL
- new net GPIO16: JP7.3, R13.2, R14.1, X1.GPIO16
- new net GPIO16EXT: JP7.2, X3-8.KL
- new net GPIO17: JP8.3, R15.2, R16.1, X1.GPIO17
- new net GPIO17EXT: JP8.2, X3-9.KL
- new net GPIO18: JP9.3, R17.2, R18.1, X1.GPIO18
- new net GPIO18EXT: JP9.2, X3-10.KL
- new net GPIO19: JP10.3, R19.2, R20.1, X1.GPIO19
- new net GPIO19EXT: JP10.2, X2-3.KL
- new net GPIO20: JP12.3, R23.2, R24.1, X1.GPIO20
- new net GPIO20EXT: JP12.2, X2-4.KL
- new net GPIO22: JP14.3, R27.2, R28.1, X1.GPIO22
- new net GPIO22EXT: JP14.2, X2-5.KL
- new net GPIO24: JP11.3, R21.2, R22.1, X1.GPIO24
- new net GPIO24EXT: JP11.2, X2-6.KL
- new net GPIO26: JP13.3, R25.2, R26.1, X1.GPIO26
- new net GPIO26EXT: JP13.2, X2-7.KL
- new net GPIO27: JP15.3, R29.2, R30.1, X1.GPIO27
- new net GPIO27EXT: JP15.2, X2-8.KL
- new net GPIO4: JP1.3, R1.2, R2.1, X1.GPIO04
- new net GPIO4EXT: JP1.2, X3-3.KL
- new net GPIO5: JP3.3, R5.2, R6.1, X1.GPIO05
- new net GPIO5EXT: JP3.2, X3-4.KL
- new net GPIO6: JP4.3, R7.2, R8.1, X1.GPIO06
- new net GPIO6EXT: JP4.2, X3-5.KL
- new net N$75: X1.GPIO21
- new net N$76: X1.SCL
- new net N$77: X1.SDA
- net 5VDC: now also X2-1.KL
