File: EasyBMS.brd (EAGLE design)
At the start: 49 x 100 mm, 149 parts, among them Q10 BSS84LT1G, Q11 BSS84LT1G, Q12 BSS84LT1G, Q13 BSS84LT1G, Q2 BSS84LT1G, Q3 BSS84LT1G, Q4 BSS84LT1G, Q5 BSS84LT1G, Q6 BSS84LT1G, Q7 BSS84LT1G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

Commit message: 8s layout is finished, its okay
Parts:
- removed C10, C11, C16, C17: 10nF, rcl:C0402
- removed LED11, LED16, LED17, LED9: KT-0603R, led:CHIPLED_0603
- removed Q12, Q13, Q6, Q7: BSS84LT1G, SamacSys_Parts:SOT96P237X111-3N
- removed R39, R43, R44, R45, R84, R85, R86, R90, R91, R92: 10R0, rcl:R1206
- removed R40, R46, R87, R93: 3.3k, rcl:R0402
- removed R41, R47, R88, R94: 470R, rcl:R0402
- removed R42, R48, R89, R95: 100R, rcl:R0402
- added R17: 0R, rcl:R0402
- added R18: 100R, rcl:R0402
- R37: value 10R0 -> 0R; device rcl:R1206 -> rcl:R0402
- R38: value 10R0 -> 100R; device rcl:R1206 -> rcl:R0402
- moved R37 27.9 mm to (27.9, 44.4), turned to 90 degrees
- moved R38 27.8 mm to (27.9, 47.5), turned to 90 degrees
Connections:
- removed net C10+: C16.2, JP7.3_C10+, Q11.2, R83.2, R84.1, R88.2
- removed net C11+: C17.2, JP7.4_C11+, Q12.2, R89.2, R90.1, R94.2
- removed net C12+: JP7.2_TOTAL+2, Q13.2, R95.2
- removed net C9+: C15.2, JP7.6_C9+, Q10.2, R76.2, R77.1, R81.2
- removed net N$33: R37.2, R38.1
- removed net N$34: R38.2, R39.1
- removed net N$35: LED9.A, Q6.3, R39.2
- removed net N$36: Q6.1, R40.2
- removed net N$37: LED9.C, R41.1
- removed net N$38: R43.2, R44.1
- removed net N$39: R44.2, R45.1
- removed net N$40: LED11.A, Q7.3, R45.2
- removed net N$41: Q7.1, R46.2
- removed net N$42: LED11.C, R47.1
- removed net N$63: R84.2, R85.1
- removed net N$64: R85.2, R86.1
- removed net N$65: LED16.A, Q12.3, R86.2
- removed net N$66: Q12.1, R87.2
- removed net N$67: LED16.C, R88.1
- removed net N$68: R90.2, R91.1
- removed net N$69: R91.2, R92.1
- removed net N$71: LED17.A, Q13.3, R92.2
- removed net N$72: Q13.1, R93.2
- removed net N$74: LED17.C, R94.1
- net C11: now also R37.1; no longer C16.1, R89.1
- net C12: now also R37.2, R38.1; no longer C17.1, R95.1
- net C4+: now also C12.2, JP7.10_C5+, JP7.5_C8+, JP7.7_C6+, JP7.8_C7+, R18.2, R49.1, R63.2; no longer C10.2, R37.1, R41.2
- net C5: now also R17.1; no longer C10.1, R42.1
- net C5+: now also C13.2, JP7.6_C9+, Q8.2, R64.2, R65.1, R69.2; no longer C11.2, JP7.10_C5+, Q6.2, R42.2, R43.1, R47.2
- net C6: now also R17.2, R18.1; no longer C11.1, R48.1
- net C6+: now also C14.2, JP7.3_C10+, Q9.2, R70.2, R71.1, R75.2; no longer C12.2, JP7.7_C6+, Q7.2, R48.2, R49.1, R63.2
- net C7+: now also C15.2, JP7.4_C11+, Q10.2, R76.2, R77.1, R81.2; no longer C13.2, JP7.8_C7+, Q8.2, R64.2, R65.1, R69.2
- net C8+: now also JP7.2_TOTAL+2, Q11.2, R38.2, R83.2; no longer C14.2, JP7.5_C8+, Q9.2, R70.2, R71.1, R75.2
- net S11: no longer R87.1
- net S12: no longer R93.1
- net S5: no longer R40.1
- net S6: no longer R46.1
Routing:
- net C11+: track 46.9 -> 0.00 mm, vias 2 -> 0
- net C9+: track 43.5 -> 0.00 mm, vias 2 -> 0
- net C10+: track 39.0 -> 0.00 mm, vias 2 -> 0
- net C4+: track 45.6 -> 80.8 mm, vias 2 -> 5
- net C12+: track 29.0 -> 0.00 mm, vias 2 -> 0
- net C6: track 28.7 -> 3.84 mm, vias 2 -> 0
- net C5: track 29.0 -> 4.22 mm, vias 2 -> 1
- net C11: track 24.6 -> 2.69 mm, vias 2 -> 0
- net C12: track 26.9 -> 5.09 mm
- net S5: track 14.9 -> 0.00 mm, vias 2 -> 0
- net S6: track 13.9 -> 0.00 mm, vias 2 -> 0
- net C8+: track 48.5 -> 36.7 mm
- net C5+: track 48.3 -> 37.3 mm, vias 2 -> 3
- net C7+: track 45.0 -> 36.0 mm
- net C6+: track 49.8 -> 42.9 mm, vias 3 -> 1
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Other:
- board text added: "8S"
