File: EasyBMS_multi.brd (EAGLE design)
At the start: 99 x 100 mm, 294 parts, among them Q10 BSS84LT1G, Q11 BSS84LT1G, Q12 BSS84LT1G, Q13 BSS84LT1G, Q2 BSS84LT1G, Q25 BSS84LT1G, Q26 BSS84LT1G, Q27 BSS84LT1G, Q28 BSS84LT1G, Q29 BSS84LT1G, Q3 BSS84LT1G, Q30 BSS84LT1G, Q31 BSS84LT1G, Q32 BSS84LT1G, Q33 BSS84LT1G, Q34 BSS84LT1G, Q35 BSS84LT1G, Q36 BSS84LT1G, Q4 BSS84LT1G, Q5 BSS84LT1G, Q6 BSS84LT1G, Q7 BSS84LT1G, Q8 BSS84LT1G, Q9 BSS84LT1G

Commit message: multiboards added
Parts:
- removed JP1, JP19: (no value), pinhead:1X13/90
- removed JP2, JP20: (no value), pinhead:1X04/90
- removed JP21: (no value), pinhead_own:1X02
- removed JP22: (no value), pinhead:2X20
- removed JP23: (no value), pinhead:1X05
- removed JP24, JP25: (no value), pinhead:1X02
- removed JP26, JP27, JP4, JP6: (no value), pinhead:2X05
- removed R173, R174: 5K1, rcl:R0603
- removed R175: 470k, rcl:R0603
- removed R176: 27K, rcl:R0603
- added H1, H2, H3, H7, H8, H9: MOUNT-HOLE3.2, holes:3,2
- added JP13: (no value), pinhead_own:1X02
- added JP14: (no value), pinhead:2X20
- added JP15: (no value), pinhead:1X05
- added JP16, JP17: (no value), pinhead:1X02
- added JP18, JP7: (no value), pinhead_own:2X11_MEB12S
- added R259, R260: 100R, rcl:R0402
- added R261, R262: 12k, rcl:R0603
- added R263, R264, R5, R6: 1k, rcl:R0603
- R177, R178: value 200R0 -> 5K1
- R179: value 200R0 -> 470k
- R180: value 200R0 -> 27K
- R181, R182: value 12k -> 200R0
- R183, R184: value 1k -> 200R0
- R185: value 100R -> 1k; device rcl:R0402 -> rcl:R0603
- R186: value 10R0 -> 1k; device rcl:R1206 -> rcl:R0603
- R187, R193, R199, R205, R211, R217, R223, R229, R235, R241, R247, R253: value 10R0 -> 100R; device rcl:R1206 -> rcl:R0402
- R189, R195, R201, R207, R213, R219, R225, R231, R237, R243, R249, R255: value 3.3k -> 10R0; device rcl:R0402 -> rcl:R1206
- R190, R196, R202, R208, R214, R220, R226, R232, R238, R244, R250, R256: value 470R -> 10R0; device rcl:R0402 -> rcl:R1206
- R191, R197, R203, R209, R215, R221, R227, R233, R239, R245, R251, R257: value 100R -> 3.3k
- R192, R198, R204, R210, R216, R222, R228, R234, R240, R246, R252: value 10R0 -> 470R; device rcl:R1206 -> rcl:R0402
- R258: value 100R -> 470R
- moved U$5 106.3 mm to (52.3, 98.0), turned to 270 degrees
- moved LED34 96.7 mm to (80.0, 97.8), turned to 0 degrees
- moved LED35 96.3 mm to (77.9, 97.8), turned to 0 degrees
- moved D6 96.2 mm to (60.4, 3.76), turned to 180 degrees
- moved LED36 96.1 mm to (75.9, 97.8), turned to 0 degrees
- moved LED33 96.1 mm to (73.9, 97.8), turned to 0 degrees
- moved C46 92.6 mm to (59.4, 6.86), turned to 180 degrees
- moved C44 91.2 mm to (66.8, 4.83), turned to 180 degrees
- moved R187 87.0 mm to (66.8, 3.56)
- moved LED38 86.9 mm to (71.8, 6.86), turned to 90 degrees
- moved R197 86.4 mm to (77.4, 7.87), turned to 90 degrees
- moved R194 86.1 mm to (60.4, 8.38), turned to 0 degrees
- moved C45 86.0 mm to (59.4, 10.4), turned to 180 degrees
- moved R196 85.9 mm to (70.6, 8.38)
- moved R193 84.9 mm to (62.4, 10.4), turned to 0 degrees
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Connections:
- removed net N$145: LED34.A, R177.1
- removed net N$146: LED35.A, R178.1
- removed net N$147: LED36.A, R179.1
- removed net N$148: LED33.A, R180.1
- removed net P10: C15.2, C54.2, JP1.10, JP19.10, Q10.2, Q33.2, R239.2, R240.1, R244.2, R76.2, R77.1, R81.2
- removed net P11: C16.2, C55.2, JP1.11, JP19.11, Q11.2, Q34.2, R245.2, R246.1, R250.2, R83.2, R84.1, R88.2
- removed net P12: C17.2, C56.2, JP1.12, JP19.12, Q12.2, Q35.2, R251.2, R252.1, R256.2, R89.2, R90.1, R94.2
- removed net P13: D2.1, D5.1, JP1.13, JP19.13, Q13.2, Q36.2, R15.2, R175.2, R257.2, R258.2, R9.2, R95.2, U$1.IN+, U$5.IN+
- removed net P2: C45.2, C7.2, D3.1, D6.1, JP1.2, JP19.2, Q2.2, Q26.2, R12.2, R14.1, R186.1, R190.2, R197.2, R23.2
- removed net P3: C47.2, C9.2, JP1.3, JP19.3, Q25.2, Q3.2, R191.2, R198.1, R202.2, R24.2, R31.1, R35.2
- removed net P4: C48.2, C8.2, JP1.4, JP19.4, Q27.2, Q5.2, R203.2, R204.1, R208.2, R25.1, R29.2, R36.2
- removed net P5: C10.2, C49.2, JP1.5, JP19.5, Q28.2, Q4.2, R209.2, R210.1, R214.2, R30.2, R37.1, R41.2
- removed net P6: C11.2, C50.2, JP1.6, JP19.6, Q29.2, Q6.2, R215.2, R216.1, R220.2, R42.2, R43.1, R47.2
- removed net P7: C12.2, C51.2, JP1.7, JP19.7, Q30.2, Q7.2, R221.2, R222.1, R226.2, R48.2, R49.1, R63.2
- removed net P8: C13.2, C52.2, JP1.8, JP19.8, Q31.2, Q8.2, R227.2, R228.1, R232.2, R64.2, R65.1, R69.2
- removed net P9: C14.2, C53.2, JP1.9, JP19.9, Q32.2, Q9.2, R233.2, R234.1, R238.2, R70.2, R71.1, R75.2
- new net C1+: C45.2, C7.2, D3.1, D6.1, JP18.16_C1+, JP7.16_C1+, Q2.2, Q26.2, R12.2, R14.1, R188.1, R192.2, R199.2, R23.2
- new net C1-: C44.2, C46.2, C5.2, C6.2, D3.2, D6.2, JP18.15_TOTAL-, JP7.15_TOTAL-, R11.2, R187.2, R194.1, R198.2, R3.2, R4.1
- new net C10+: C16.2, C55.2, JP18.3_C10+, JP7.3_C10+, Q11.2, Q34.2, R247.2, R248.1, R252.2, R83.2, R84.1, R88.2
- new net C11+: C17.2, C56.2, JP18.4_C11+, JP7.4_C11+, Q12.2, Q35.2, R253.2, R254.1, R258.2, R89.2, R90.1, R94.2
- new net C12+: JP18.2_TOTAL+2, JP7.2_TOTAL+2, Q13.2, Q36.2, R259.2, R95.2
- new net C2+: C47.2, C9.2, JP18.13_C2+, JP7.13_C2+, Q25.2, Q3.2, R193.2, R200.1, R204.2, R24.2, R31.1, R35.2
- new net C3+: C48.2, C8.2, JP18.14_C3+, JP7.14_C3+, Q27.2, Q5.2, R205.2, R206.1, R210.2, R25.1, R29.2, R36.2
- new net C4+: C10.2, C49.2, JP18.11_C4+, JP7.11_C4+, Q28.2, Q4.2, R211.2, R212.1, R216.2, R30.2, R37.1, R41.2
- new net C5+: C11.2, C50.2, JP18.10_C5+, JP7.10_C5+, Q29.2, Q6.2, R217.2, R218.1, R222.2, R42.2, R43.1, R47.2
- new net C6+: C12.2, C51.2, JP18.7_C6+, JP7.7_C6+, Q30.2, Q7.2, R223.2, R224.1, R228.2, R48.2, R49.1, R63.2
- new net C7+: C13.2, C52.2, JP18.8_C7+, JP7.8_C7+, Q31.2, Q8.2, R229.2, R230.1, R234.2, R64.2, R65.1, R69.2
- new net C8+: C14.2, C53.2, JP18.5_C8+, JP7.5_C8+, Q32.2, Q9.2, R235.2, R236.1, R240.2, R70.2, R71.1, R75.2
- new net C9+: C15.2, C54.2, JP18.6_C9+, JP7.6_C9+, Q10.2, Q33.2, R241.2, R242.1, R246.2, R76.2, R77.1, R81.2
- new net N$15: R6.1, U$2.JP1.7
- new net N$253: R255.2, R256.1
- new net N$254: LED48.A, Q36.3, R256.2
- new net N$255: Q36.1, R257.2
- new net N$256: LED48.C, R258.1
- new net N$257: R263.1, U$6.JP1.4
- new net N$258: R264.1, U$6.JP1.7
- new net N$7: R5.1, U$2.JP1.4
- new net VIN: D2.1, D5.1, JP18.1_TOTAL+, JP7.1_TOTAL+, R15.2, R179.2, R260.2, R9.2, U$1.IN+, U$5.IN+
- net 5VDC: now also JP14.10, JP15.1, JP15.2, R177.2, R178.2; no longer JP22.10, JP23.1, JP23.2, R173.2, R174.2
- net A0IN: now also R179.1, R180.2; no longer R175.1, R176.2
- net C0: now also JP14.30, R187.1; no longer JP22.30, R185.1
- net C1: now also JP14.34, R199.1; no longer JP22.34, JP27.9, JP6.9, R197.1
- net C10: now also JP14.11, R247.1; no longer JP22.11, JP26.3, JP4.3, R245.1
- net C11: now also JP14.7, R253.1; no longer JP22.7, JP26.1, JP4.1, R251.1
- net C12: now also JP14.3, R259.1; no longer JP22.3, JP26.10, JP26.2, JP26.4, JP26.6, JP26.8, JP4.10, JP4.2, JP4.4, JP4.6, JP4.8, R257.1
- net C2: now also JP14.38, R193.1; no longer JP22.38, JP27.7, JP6.7, R191.1
- net C3: now also JP14.39, R205.1; no longer JP22.39, JP27.5, JP6.5, R203.1
- net C4: now also JP14.35, R211.1; no longer JP22.35, JP27.3, JP6.3, R209.1
- net C5: now also JP14.31, R217.1; no longer JP22.31, JP27.1, JP6.1, R215.1
- net C6: now also JP14.27, R223.1; no longer JP22.27, JP27.10, JP27.2, JP27.4, JP27.6, JP27.8, JP6.10, JP6.2, JP6.4, JP6.6, JP6.8, R221.1
- net C7: now also JP14.23, R229.1; no longer JP22.23, JP26.9, JP4.9, R227.1
- net C8: now also JP14.19, R235.1; no longer JP22.19, JP26.7, JP4.7, R233.1
- net C9: now also JP14.15, R241.1; no longer JP22.15, JP26.5, JP4.5, R239.1
- net CSB: now also JP14.8, R264.2, R6.2; no longer JP22.8, U$2.JP1.7, U$6.JP1.7
- net GND: now also JP14.16, JP14.18, JP15.4, JP15.5, JP16.1, JP16.2, JP17.1, JP17.2, JP18.17_TOTAL-, JP7.17_TOTAL-, R180.1, R261.1, R262.1; no longer C44.2, C46.2, C5.2, C6.2, D3.2, D6.2, JP1.1, JP19.1, JP22.16, JP22.18, JP23.4, JP23.5, JP24.1, JP24.2, JP25.1, JP25.2, R11.2, R176.1, R181.1, R182.1, R185.2, R192.1, R196.2, R3.2, R4.1
- net GPIO4: now also JP14.22; no longer JP22.22
- net GPIO5: now also JP14.20; no longer JP22.20
- net ISIGNAL: now also JP14.24, JP15.3; no longer JP22.24, JP23.3
- net MISO: now also JP14.2, R178.1, R185.2; no longer JP22.2, R174.1, R183.2
- net MOSI: now also JP14.4, R177.1, R186.2; no longer JP22.4, R173.1, R184.2
- net N$149: now also LED34.A, R181.1; no longer R177.2, U$6.JP2.3
- net N$150: now also LED35.A, R182.1; no longer R180.2, U$6.JP2.6
- net N$151: now also LED36.A, R183.1; no longer R179.2, U$6.JP2.5
- net N$152: now also LED33.A, R184.1; no longer R178.2, U$6.JP2.4
- net N$153: now also R181.2, U$6.JP2.3; no longer R183.1, U$6.JP1.5
- net N$154: now also R184.2, U$6.JP2.6; no longer R184.1, U$6.JP1.6
- net N$155: now also R183.2, U$6.JP2.5; no longer JP21.2, U$6.JP1.1
- net N$156: now also R182.2, U$6.JP2.4; no longer JP21.1, U$6.JP1.3
- net N$157: now also R185.1, U$6.JP1.5; no longer R186.2, R187.1
- net N$158: now also R186.1, U$6.JP1.6; no longer R187.2, R188.1
- net N$159: now also JP13.2, U$6.JP1.1; no longer LED37.A, Q25.3, R188.2
- net N$160: now also JP13.1, U$6.JP1.3; no longer Q25.1, R189.2
- net N$161: now also R188.2, R189.1; no longer LED37.C, R190.1
- net N$162: now also R189.2, R190.1; no longer R192.2, R193.1
- net N$163: now also LED37.A, Q25.3, R190.2; no longer R193.2, R194.1
- net N$164: now also Q25.1, R191.2; no longer LED38.A, Q26.3, R194.2
- net N$165: now also LED37.C, R192.1; no longer Q26.1, R195.2
- net N$166: now also R194.2, R195.1; no longer LED38.C, R196.1
- net N$167: now also R195.2, R196.1; no longer R198.2, R199.1
- net N$168: now also LED38.A, Q26.3, R196.2; no longer R199.2, R200.1
- net N$169: now also Q26.1, R197.2; no longer LED39.A, Q27.3, R200.2
- net N$170: now also LED38.C, R198.1; no longer Q27.1, R201.2
- net N$171: now also R200.2, R201.1; no longer LED39.C, R202.1
- net N$172: now also R201.2, R202.1; no longer R204.2, R205.1
- net N$173: now also LED39.A, Q27.3, R202.2; no longer R205.2, R206.1
- net N$174: now also Q27.1, R203.2; no longer LED40.A, Q28.3, R206.2
- net N$175: now also LED39.C, R204.1; no longer Q28.1, R207.2
- net N$176: now also R206.2, R207.1; no longer LED40.C, R208.1
- net N$177: now also R207.2, R208.1; no longer R210.2, R211.1
- net N$178: now also LED40.A, Q28.3, R208.2; no longer R211.2, R212.1
- net N$179: now also Q28.1, R209.2; no longer LED41.A, Q29.3, R212.2
- net N$180: now also LED40.C, R210.1; no longer Q29.1, R213.2
- net N$181: now also R212.2, R213.1; no longer LED41.C, R214.1
- net N$182: now also R213.2, R214.1; no longer R216.2, R217.1
- net N$183: now also LED41.A, Q29.3, R214.2; no longer R217.2, R218.1
- net N$184: now also Q29.1, R215.2; no longer LED42.A, Q30.3, R218.2
- net N$185: now also LED41.C, R216.1; no longer Q30.1, R219.2
- net N$186: now also R218.2, R219.1; no longer LED42.C, R220.1
- net N$187: now also R219.2, R220.1; no longer R222.2, R223.1
- net N$188: now also LED42.A, Q30.3, R220.2; no longer R223.2, R224.1
- net N$189: now also Q30.1, R221.2; no longer LED43.A, Q31.3, R224.2
- net N$190: now also LED42.C, R222.1; no longer Q31.1, R225.2
- net N$191: now also R224.2, R225.1; no longer LED43.C, R226.1
- net N$192: now also R225.2, R226.1; no longer R228.2, R229.1
- net N$193: now also LED43.A, Q31.3, R226.2; no longer R229.2, R230.1
- net N$194: now also Q31.1, R227.2; no longer LED44.A, Q32.3, R230.2
- net N$195: now also LED43.C, R228.1; no longer Q32.1, R231.2
- net N$196: now also R230.2, R231.1; no longer LED44.C, R232.1
- net N$197: now also R231.2, R232.1; no longer R234.2, R235.1
- net N$198: now also LED44.A, Q32.3, R232.2; no longer R235.2, R236.1
- net N$199: now also Q32.1, R233.2; no longer LED45.A, Q33.3, R236.2
- net N$200: now also LED44.C, R234.1; no longer Q33.1, R237.2
- net N$201: now also R236.2, R237.1; no longer LED45.C, R238.1
- net N$205: now also R237.2, R238.1; no longer R240.2, R241.1
- net N$239: now also LED45.A, Q33.3, R238.2; no longer R241.2, R242.1
- net N$240: now also Q33.1, R239.2; no longer LED46.A, Q34.3, R242.2
- net N$241: now also LED45.C, R240.1; no longer Q34.1, R243.2
- net N$242: now also R242.2, R243.1; no longer LED46.C, R244.1
- net N$243: now also R243.2, R244.1; no longer R246.2, R247.1
- net N$244: now also LED46.A, Q34.3, R244.2; no longer R247.2, R248.1
- net N$245: now also Q34.1, R245.2; no longer LED47.A, Q35.3, R248.2
- net N$246: now also LED46.C, R246.1; no longer Q35.1, R249.2
- net N$247: now also R248.2, R249.1; no longer LED47.C, R250.1
- net N$248: now also R249.2, R250.1; no longer R252.2, R253.1
- net N$249: now also LED47.A, Q35.3, R250.2; no longer R253.2, R254.1
- net N$250: now also Q35.1, R251.2; no longer LED48.A, Q36.3, R254.2
- net N$251: now also LED47.C, R252.1; no longer Q36.1, R255.2
- net N$252: now also R254.2, R255.1; no longer LED48.C, R256.1
- net S1: now also JP14.32, R197.1; no longer JP22.32, R195.1
- net S10: now also JP14.13, R245.1; no longer JP22.13, R243.1
- net S11: now also JP14.9, R251.1; no longer JP22.9, R249.1
- net S12: now also JP14.5, R257.1; no longer JP22.5, R255.1
- net S2: now also JP14.36, R191.1; no longer JP22.36, R189.1
- net S3: now also JP14.40, R203.1; no longer JP22.40, R201.1
- net S4: now also JP14.37, R209.1; no longer JP22.37, R207.1
- net S5: now also JP14.33, R215.1; no longer JP22.33, R213.1
- net S6: now also JP14.29, R221.1; no longer JP22.29, R219.1
- net S7: now also JP14.25, R227.1; no longer JP22.25, R225.1
- net S8: now also JP14.21, R233.1; no longer JP22.21, R231.1
- net S9: now also JP14.17, R239.1; no longer JP22.17, R237.1
- net SCK: now also JP14.6, R263.2, R5.2; no longer JP22.6, U$2.JP1.4, U$6.JP1.4
- net V+: now also JP14.1, R260.1; no longer JP22.1, R258.1
- net VREF1: now also JP14.12; no longer JP22.12
- net VREF2: now also JP14.14, JP18.19_THERMO1_IN, JP18.20_THERMO2_IN, JP7.19_THERMO1_IN, JP7.20_THERMO2_IN; no longer JP2.1, JP2.3, JP20.1, JP20.3, JP22.14
- net VTEMP1: now also JP14.28, JP18.21_THERMO1_OUT, JP7.21_THERMO1_OUT, R261.2; no longer JP2.2, JP20.2, JP22.28, R181.2
- net VTEMP2: now also JP14.26, JP18.22_THERMO2_OUT, JP7.22_THERMO2_OUT, R262.2; no longer JP2.4, JP20.4, JP22.26, R182.2
Routing:
- net P13: track 297.0 -> 0.00 mm, vias 6 -> 0
- net VIN: track 0.00 -> 196.4 mm, vias 0 -> 4
- net C1+: track 0.00 -> 97.9 mm, vias 0 -> 8
- net GND: track 130.2 -> 34.5 mm, vias 188 -> 328
- net C3+: track 0.00 -> 91.6 mm, vias 0 -> 6
- net C2+: track 0.00 -> 87.9 mm, vias 0 -> 6
- net C4+: track 0.00 -> 85.6 mm, vias 0 -> 6
- net C11+: track 0.00 -> 84.8 mm, vias 0 -> 6
- net C7+: track 0.00 -> 84.5 mm, vias 0 -> 6
- net C5+: track 0.00 -> 82.7 mm, vias 0 -> 6
- net C9+: track 0.00 -> 82.1 mm, vias 0 -> 6
- net C6+: track 0.00 -> 81.6 mm, vias 0 -> 6
- net C8+: track 0.00 -> 78.8 mm, vias 0 -> 4
- net C10+: track 0.00 -> 78.0 mm, vias 0 -> 4
- net C1: track 140.1 -> 62.5 mm, vias 4 -> 2
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Other:
- board text added: "EasyBMS MEB12S v1.1 13.12.2021"
