File: MEB-Version(12S&8S)/EasyBMS.kicad_sch (KiCad schematic)
At the start: 174 parts, among them IC1 XL7046, IC2 LTC6811IG-1#PBF, IC3 ISO1042DWV, IC4 AMS1117-3.3, J1 TYPE-C-31-M-12, Q14 CJ2301, Q15 CJ2301, Q16 CJ2301, Q18 CJ2301, Q20 CJ2301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

Commit message: change to correct footprints, add LCSC numbers to schematic
Parts:
- C1, C13, C19, C4, C5, C7: LCSC (none) -> C52923
- C10, C11, C15, C17, C3: LCSC (none) -> C307331
- C12: LCSC (none) -> C96123
- C14: LCSC (none) -> C16780
- C16, C9: LCSC (none) -> C1548
- C20, C21: LCSC (none) -> C28233
- C23, C25, C28, C29, C31, C33, C35, C37, C39, C41, C43, C45, C47, C6: LCSC (none) -> C15195
- C27: LCSC (none) -> C15849
- C8: LCSC (none) -> C59461
- IC2: LCSC (none) -> C689566
- LED2: LCSC (none) -> C5349954
- R1: LCSC (none) -> C22775
- R10, R11: LCSC (none) -> C25905
- R100, R101, R104, R105, R112, R113, R120, R121, R128, R129, R136, R137, R144, R145, R152, R153, R160, R161, R168, R169, R176, R177, R82, R96: LCSC (none) -> C17903
- R102, R106, R114, R122, R130, R138, R146, R154, R162, R170, R178, R55, R97: LCSC (none) -> C25890
- R103, R107, R115, R123, R131, R139, R147, R155, R163, R171, R179, R60, R9, R98: LCSC (none) -> C25076
- R12: LCSC (none) -> C25079
- R13, R14, R2, R21, R6: LCSC (none) -> C25744
- R15: footprint EasyBMS:R0402_334 -> EasyBMS:R0603_334; LCSC (none) -> C23178
- R16: footprint EasyBMS:R0402_334 -> EasyBMS:R0603_334; LCSC (none) -> C22967
- R17: LCSC (none) -> C4184
- R19: LCSC (none) -> C17901
- R20: LCSC (none) -> C7250
- R3, R7: LCSC (none) -> C25804
- R57, R58: LCSC (none) -> C25752

Commit message: fixed wrong footprints and symbols, connect 3d models with footprints
Connections:
- net GND: no longer IC1.9 (EP), J1.S2 (SHIELD), J1.S3 (SHIELD), J1.S4 (SHIELD)
- net at D3.C, IC1.5 (SW), L1.P$1 (1): now also IC1.9 (SW)
Changed lines of the file:
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@@
 	)
 	(junction
-		(at 299.72 68.58)
-		(diameter 0)
-		(color 0 0 0 0)
-	)
-	(junction
 		(at 176.53 242.57)
 		(diameter 0)
@@
 	(wire
 		(pts
-			(xy 304.8 68.58) (xy 299.72 68.58)
+			(xy 294.64 68.58) (xy 304.8 68.58)
 		)
 		(stroke
@@
 	(wire
 		(pts
-			(xy 299.72 60.96) (xy 299.72 68.58)
-		)
-		(stroke
-			(width 0.1524)
-			(type solid)
-		)
-	)
-	(wire
-		(pts
 			(xy 166.37 445.77) (xy 314.96 445.77)
 		)
@@
 	(wire
 		(pts
-			(xy 299.72 68.58) (xy 294.64 68.58)
-		)
-		(stroke
-			(width 0.1524)
-			(type solid)
-		)
-	)
-	(wire
-		(pts
 			(xy 495.3 203.2) (xy 501.65 203.2)
 		)
@@
 			)
 		)
-		(property "Description" ""
+		(property "Description" "https://pricing.snapeda.com/parts/TYPE-C-31-M-12/HRO%20Electronics%20Co.%2C%20Ltd./view-part?ref=eda Check availability"
 			(at 290.83 140.97 0)
 			(effects
@@
 		(pin "S1"
 		)
-		(pin "S4"
-		)
 		(pin "A6"
 		)
@@
 		(pin "B5"
 		)
-		(pin "S2"
-		)
-		(pin "S3"
-		)
 		(pin "A1_B12"
 		)
@@
 			)
 		)
-		(property "Description" ""
+		(property "Description" "XL7046 1.0A 100KHz 90V Buck DC to DC Converter\n\nGeneral Description The XL7046 is a 100KHz fixed frequency PWM buck (step-down) DC/DC converter, capable of driving a 1.0A load with high efficiency, low ripple and excellent line and load regulation. Requiring a minimum number of external components, the regulator is simple to use and include internal frequency compensation and a fixed-frequency oscillator.   Datasheet"
 			(at 271.78 40.64 0)
 			(effects
@@
 		(pin "8"
 		)
-		(pin "9"
-		)
 		(pin "4"
 		)
+		(pin "9"
+		)
 		(instances
 			(project ""
@@
 			)
 		)
-		(property "Description" ""
+		(property "Description" "800mA and 1A Low Dropout (LDO) Positive Regulator\n\n1.8V, 2.5V, 2.85V, 3.3V, 5V, and Adj"
 			(at 417.83 102.87 0)
 			(effects
@@
 		(pin "1"
 		)
+		(pin "4"
+		)
 		(instances
