File: Dual-Version/call_pack_1.kicad_sch (KiCad schematic)
At the start: 121 parts, among them IC2 LTC6811IG-1#PBF, J2 RJ45_Shielded, J3 RJ45_Shielded, Q14 CJ2301, Q15 CJ2301, Q16 CJ2301, Q18 CJ2301, Q20 CJ2301, Q22 CJ2301, Q24 CJ2301, Q26 CJ2301, Q28 CJ2301, Q30 CJ2301, Q32 CJ2301, Q34 CJ2301

Commit message: schematic improvements, parts changed, layout progress
Parts:
- removed C12+POWER2: SJ, EasyBMS:SJ_252, symbol EasyBMS-eagle-import:SJ
- removed C18: 10nF, symbol Device:C
- removed J2, J3: RJ45_Shielded, symbol Connector:RJ45_Shielded
- removed R1, R22: 49R9, EasyBMS:R0603_334, symbol EasyBMS-eagle-import:R-EU_R0603
- removed R59: 600R@100MHz, EasyBMS:R1206_334, symbol EasyBMS-eagle-import:R-EU_R1206
- IC2: value LTC6811IG-1#PBF -> LTC6811IG-1
- renumbered C1-/GND to GND2
Connections:
- net GND: now also GND2.1; no longer IC2.40 (ISOMD)
- net VTEMP1: now also IC2.29 (GPIO3); no longer IC2.28 (GPIO2)
- net VTEMP2: now also IC2.28 (GPIO2); no longer IC2.29 (GPIO3)
- net DRIVE: now reaches IC2.38 (DRIVE)
- net +5V renamed VREG
- net CSLTC renamed CSBIMA
- net CURRENT_SENSE renamed CURRENTSENSE
- net MISO renamed SDO
- net MOSI renamed SDI
- net SCLK renamed SCKIPA
- new net ISOMD: IC2.40 (ISOMD)
- no-connect marks 0 -> 4
Other:
- moved on the sheet: C1, C19, C20, C4, IC2, R17, R23, R57, R58, R9

Commit message: schematic and layout finalized, production data generated
Parts:
- D10, D12, D14, D16, D18, D20, D22, D24, D4, D5, D6, D8, GND2, IC2, JP10, JP11, JP12, JP13, JP2, JP3, JP4, JP5, JP6, JP8, JP9: now left out of the parts list
- R17, R23: LCSC (none) -> C21190
Changed lines of the file:
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@@
 		(polyline
 			(pts
-				(xy 81.28 347.98) (xy 194.31 347.98) (xy 194.31 322.58) (xy 81.28 322.58)
+				(xy 81.28 292.1) (xy 194.31 292.1) (xy 194.31 266.7) (xy 81.28 266.7)
 			)
 			(stroke
@@
 		(polyline
 			(pts
-				(xy 81.28 152.4) (xy 194.31 152.4) (xy 194.31 127) (xy 81.28 127)
+				(xy 22.86 16.51) (xy 408.94 17.78) (xy 409.0193 403.7806) (xy 12.7 400.05) (xy 12.7 26.67)
 			)
 			(stroke
@@
 		(polyline
 			(pts
-				(xy 81.28 264.16) (xy 194.31 264.16) (xy 194.31 238.76) (xy 81.28 238.76)
+				(xy 81.28 68.58) (xy 194.31 68.58) (xy 194.31 43.18) (xy 81.28 43.18)
 			)
 			(stroke
@@
 		(polyline
 			(pts
-				(xy 81.28 96.52) (xy 194.31 96.52) (xy 194.31 71.12) (xy 81.28 71.12)
+				(xy 81.28 236.22) (xy 194.31 236.22) (xy 194.31 210.82) (xy 81.28 210.82)
 			)
 			(stroke
@@
 		(polyline
 			(pts
-				(xy 81.28 292.1) (xy 194.31 292.1) (xy 194.31 266.7) (xy 81.28 266.7)
+				(xy 81.28 320.04) (xy 194.31 320.04) (xy 194.31 294.64) (xy 81.28 294.64)
 			)
 			(stroke
@@
 		(polyline
 			(pts
-				(xy 81.28 236.22) (xy 194.31 236.22) (xy 194.31 210.82) (xy 81.28 210.82)
+				(xy 81.28 180.34) (xy 194.31 180.34) (xy 194.31 154.94) (xy 81.28 154.94)
 			)
 			(stroke
@@
 		(polyline
 			(pts
-				(xy 81.28 124.46) (xy 194.31 124.46) (xy 194.31 99.06) (xy 81.28 99.06)
+				(xy 81.28 208.28) (xy 194.31 208.28) (xy 194.31 182.88) (xy 81.28 182.88)
 			)
 			(stroke
@@
 		(polyline
 			(pts
-				(xy 22.86 16.51) (xy 408.94 17.78) (xy 409.0193 403.7806) (xy 12.7 400.05) (xy 12.7 26.67)
+				(xy 81.28 264.16) (xy 194.31 264.16) (xy 194.31 238.76) (xy 81.28 238.76)
 			)
 			(stroke
@@
 		(polyline
 			(pts
-				(xy 81.28 208.28) (xy 194.31 208.28) (xy 194.31 182.88) (xy 81.28 182.88)
+				(xy 81.28 96.52) (xy 194.31 96.52) (xy 194.31 71.12) (xy 81.28 71.12)
 			)
 			(stroke
@@
 		(polyline
 			(pts
-				(xy 81.28 375.92) (xy 194.31 375.92) (xy 194.31 350.52) (xy 81.28 350.52)
+				(xy 81.28 152.4) (xy 194.31 152.4) (xy 194.31 127) (xy 81.28 127)
 			)
 			(stroke
@@
 		(polyline
 			(pts
-				(xy 81.28 68.58) (xy 194.31 68.58) (xy 194.31 43.18) (xy 81.28 43.18)
+				(xy 81.28 124.46) (xy 194.31 124.46) (xy 194.31 99.06) (xy 81.28 99.06)
 			)
 			(stroke
@@
 		(polyline
 			(pts
-				(xy 81.28 320.04) (xy 194.31 320.04) (xy 194.31 294.64) (xy 81.28 294.64)
+				(xy 81.28 375.92) (xy 194.31 375.92) (xy 194.31 350.52) (xy 81.28 350.52)
 			)
 			(stroke
@@
 		(polyline
 			(pts
-				(xy 81.28 180.34) (xy 194.31 180.34) (xy 194.31 154.94) (xy 81.28 154.94)
+				(xy 81.28 347.98) (xy 194.31 347.98) (xy 194.31 322.58) (xy 81.28 322.58)
 			)
 			(stroke
@@
 		(unit 1)
 		(exclude_from_sim no)
-		(in_bom yes)
+		(in_bom no)
 		(on_board yes)
 		(dnp no)
@@
 		(unit 1)
 		(exclude_from_sim no)
-		(in_bom yes)
+		(in_bom no)
 		(on_board yes)
 		(dnp no)
@@
 		(unit 1)
 		(exclude_from_sim no)
-		(in_bom yes)
+		(in_bom no)
 		(on_board yes)
 		(dnp no)
@@
 		(unit 1)
 		(exclude_from_sim no)
-		(in_bom yes)
+		(in_bom no)
 		(on_board yes)
 		(dnp no)
@@
 		(unit 1)
 		(exclude_from_sim no)
-		(in_bom yes)
+		(in_bom no)
 		(on_board yes)
 		(dnp no)
@@
 		(unit 1)
 		(exclude_from_sim no)
-		(in_bom yes)
+		(in_bom no)
 		(on_board yes)
 		(dnp no)
@@
 		(unit 1)
 		(exclude_from_sim no)
-		(in_bom yes)
+		(in_bom no)
 		(on_board yes)
 		(dnp no)
@@
 		(unit 1)
 		(exclude_from_sim no)
-		(in_bom yes)
+		(in_bom no)
 		(on_board yes)
 		(dnp no)
@@
 			)
 		)
-		(property "LCSC" ""
+		(property "LCSC" "C21190"
 			(at 495.3 217.17 0)
 			(effects
@@
 		(unit 1)
 		(exclude_from_sim no)
-		(in_bom yes)
+		(in_bom no)
 		(on_board yes)
 		(dnp no)
@@
 		(unit 1)
 		(exclude_from_sim no)
-		(in_bom yes)
+		(in_bom no)
 		(on_board yes)
 		(dnp no)
@@
 		(unit 1)
 		(exclude_from_sim no)
-		(in_bom yes)
+		(in_bom no)
 		(on_board yes)
 		(dnp no)
@@
 		(unit 1)
 		(exclude_from_sim no)
-		(in_bom yes)
+		(in_bom no)
 		(on_board yes)
 		(dnp no)
@@
 		(unit 1)
 		(exclude_from_sim no)
-		(in_bom yes)
+		(in_bom no)
 		(on_board yes)
 		(dnp no)
@@
 		(unit 1)
 		(exclude_from_sim no)
-		(in_bom yes)
+		(in_bom no)
 		(on_board yes)
 		(dnp no)
@@
 		(unit 1)
 		(exclude_from_sim no)
-		(in_bom yes)
+		(in_bom no)
 		(on_board yes)
 		(dnp no)
@@
 		(unit 1)
 		(exclude_from_sim no)
-		(in_bom yes)
+		(in_bom no)
 		(on_board yes)
 		(dnp no)
@@
 		(unit 1)
 		(exclude_from_sim no)
-		(in_bom yes)
+		(in_bom no)
 		(on_board yes)
 		(dnp no)
@@
 		(unit 1)
 		(exclude_from_sim no)
-		(in_bom yes)
+		(in_bom no)
 		(on_board yes)
 		(dnp no)
@@
 		(unit 1)
 		(exclude_from_sim no)
-		(in_bom yes)
+		(in_bom no)
 		(on_board yes)
 		(dnp no)
@@
 			)
 		)
-		(property "LCSC" ""
+		(property "LCSC" "C21190"
 			(at 481.33 217.17 0)
 			(effects
@@
 		(unit 1)
 		(exclude_from_sim no)
-		(in_bom yes)
+		(in_bom no)
 		(on_board yes)
 		(dnp no)
@@
 		(unit 1)
 		(exclude_from_sim no)
-		(in_bom yes)
+		(in_bom no)
 		(on_board yes)
 		(dnp no)
@@
 		(unit 1)
 		(exclude_from_sim no)
-		(in_bom yes)
+		(in_bom no)
 		(on_board yes)
 		(dnp no)
@@
 		(unit 1)
 		(exclude_from_sim no)
-		(in_bom yes)
+		(in_bom no)
 		(on_board yes)
 		(dnp no)
@@
 		(unit 1)
 		(exclude_from_sim no)
-		(in_bom yes)
+		(in_bom no)
 		(on_board yes)
 		(dnp no)
@@
 		(unit 1)
 		(exclude_from_sim no)
-		(in_bom yes)
+		(in_bom no)
 		(on_board yes)
 		(dnp no)
