File: Dual-Version/EasyBMS.kicad_sch (KiCad schematic)
At the start: 82 parts, among them IC1 XL7046, IC3 ISO1042DWV, IC4 AMS1117-3.3, IC6 AMS1117-5, J1 TYPE-C-31-M-12, J6 RJ45_Shielded, J7 RJ45_Shielded, J8 RJ45_Shielded, U1 ESP32-C6-MINI-1-N4, U2 ACS770xCB-100B-PFF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

Commit message: schematic improvements, parts changed, layout progress
Parts:
- removed C12: 47µF, EasyBMS:C1206_334, symbol EasyBMS-eagle-import:C-EUC1206
- removed C2: 100µF/16V, EasyBMS:153CLV-0605_334, symbol EasyBMS-eagle-import:CPOL-EU153CLV-0605
- removed C60, C7: 1uF, EasyBMS:C0402_334, symbol EasyBMS-eagle-import:C-EUC0402
- removed C63: 22uF, EasyBMS:C0603_334, symbol EasyBMS-eagle-import:C-EUC0603
- removed IC3: ISO1042DWV, EasyBMS:SOIC127P1150X280-8N, symbol EasyBMS-eagle-import:ISO1042DWV
- removed J6, J7, J8: RJ45_Shielded, symbol Connector:RJ45_Shielded
- removed R61: 600R@100MHz, EasyBMS:R1206_334, symbol EasyBMS-eagle-import:R-EU_R1206
- added C12, C18, C64, C65, C7: 22uF, EasyBMS:C0805_334, symbol EasyBMS-eagle-import:C-EUC0603
- added C2: 10uF, Capacitor_SMD:C_0805_2012Metric, symbol Device:C
- added C56, C66: 10nF, EasyBMS:C0402_334, symbol EasyBMS-eagle-import:C-EUC0402
- added C59: 100nF, EasyBMS:C0805_334, symbol EasyBMS-eagle-import:C-EUC0805
- added CAN-GNDP1, CAN-GNDV1, CAN-HP1, CAN-HV1, CAN-LP1, CAN-LV1, RS485-AP1, RS485-BP1, RS485-GNDPWR1, RS485-VDD1: SJ, EasyBMS:SJ_252, symbol EasyBMS-eagle-import:SJ
- added J2: Screw_Terminal_01x04, TerminalBlock_TE-Connectivity:TerminalBlock_TE_282834-4_1x04_P2.54mm_Horizontal, symbol Connector:Screw_Terminal_01x04
- added Q13: NSV1C201MZ4, Package_TO_SOT_SMD:SOT-223, symbol Transistor_BJT:BCP56
- added R1, R22, R92, R93: 49R9, EasyBMS:R0603_334, symbol EasyBMS-eagle-import:R-EU_R0603
- added R59: 100R, EasyBMS:R1206_334, symbol EasyBMS-eagle-import:R-EU_R1206
- added R90: 100R, EasyBMS:R0603_334, symbol EasyBMS-eagle-import:R-EU_R0603
- added U4, U6: RJ-064-1, RJ45 Connectors:CONN-SMD_RJ-064, symbol RJ45 Connectors:RJ-064-1
- added U5: CA-IS3050CG, Package_SO:SOIC-8_7.5x5.85mm_P1.27mm, symbol Interface_CAN_LIN:ISO1050DUB
- added U7: TME-0305S, Converter_DCDC:Converter_DCDC_TRACO_TME_03xxS_05xxS_12xxS_Single_THT, symbol Converter_DCDC:TME-0305S
- B1: footprint Meine BE:RS-485-MODULE -> RS485 Modul:RS-485-MODULE; symbol Meine BE:RS-485-MODULE -> RS485 Modul:RS-485-MODULE
- H4, H5: footprint MountingHole:MountingHole_8.4mm_M8_Pad_Via -> MountingHole:MountingHole_6.5mm_Pad_Via
- R24: value 4k7 -> 10k
- renumbered IP-/GND to IP-/GND1
Connections:
- net +12V: now also C65.1, C7.1, U4.2
- net +3V3: now also C2.1, U5.1 (VCC1), U7.2 (+Vin)
- net +5V: now also C12.1
- net Cell Pack 1/IMB: now also R22.1
- net Cell Pack 1/IPB: now also R1.2
- net Cell Pack 2/C12+POWER: now also R59.1
- net GND: now also IP-/GND1.1, C12.2, C2.2, C66.2, C7.2, U5.4 (GND1), U7.1 (-Vin)
- net GNDPWR: now also C64.2, C65.2, RS485-GNDPWR1.2, U4.10 (EH), U4.11 (EH), U4.12 (EH), U4.3, U4.9 (EH)
- net VDD: now also C64.1, RS485-VDD1.1
- net at C11.1, D37.1 (K): now also C18.1, J2.1 (Pin_1), RS485-VDD1.2, U5.8 (VCC2), U7.4 (+Vout)
- net at C11.2, D35.1 (A1), D36.1 (A1)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: now also C18.2, CAN-GNDP1.2, CAN-GNDV1.2, J2.4 (Pin_4), RS485-GNDPWR1.1, U5.5 (GND2), U6.10 (EH), U6.11 (EH), U6.12 (EH), U6.9 (EH), U7.3 (-Vout)
- net at U1.28 (IO22): now also U5.2 (RXD)
- net at U1.29 (IO23): now also U5.3 (TXD)
- net at D35.2 (A2), D38.1 (A1), F2.1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: now also U5.6 (CANL)
- net at D36.2 (A2), D38.2 (A2), F1.1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: now also U5.7 (CANH)
- net at B1.A+: now also RS485-AP1.1, U4.4
- net at B1.B-: now also RS485-BP1.1, U4.5
- net at F2.2: now also CAN-LP1.2, CAN-LV1.2, J2.3 (Pin_3)
- net at F1.2: now also CAN-HP1.2, CAN-HV1.2, J2.2 (Pin_2)
- net Cell Pack 1/CURRENT_SENSE renamed Cell Pack 1/CURRENTSENSE
- net Cell Pack 2/IMA renamed Cell Pack 2/CSBIMA
- net Cell Pack 2/CSBIMA: now also R93.1
- net Cell Pack 2/IPA renamed Cell Pack 2/SCKIPA
- net Cell Pack 2/SCKIPA: now also R92.2
- new net: CAN-GNDV1.1, U6.3
- new net: CAN-HP1.1, U6.4
- new net: CAN-LP1.1, U6.5
- new net: CAN-GNDP1.1, U6.6
- new net: CAN-HV1.1, RS485-AP1.2, U6.7
- new net: CAN-LV1.1, RS485-BP1.2, U6.8
- new net: C66.1, R1.1, R22.2
- new net: C59.2, Q13.2 (C), R59.2
- new net: C56.1, R92.1, R93.2
- new net Cell Pack 2/IMB: R90.2
- new net Cell Pack 2/IPB: R90.1
- new net DRIVE2: Q13.1 (B)
- new net GND1: C56.2, C59.1
- new net VREG2: Q13.3 (E)
- no-connect marks 10 -> 12
Other:
- sheet Cell Pack 1 ports: added CSBIMA, CURRENTSENSE, DRIVE, ISOMD, SCKIPA, SDI, SDO, VREG; removed CURRENT_SENSE
- sheet Cell Pack 2 ports: added CSBIMA, CURRENTSENSE, DRIVE, IMB, IPB, ISOMD, SCKIPA, SDI, SDO, VREG; removed CURRENT_SENSE, IMA, IPA
- moved on the sheet: C10, C11, C22, C42, C57, C58, D35, D36, D37, D38, F1, F2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

Commit message: schematic and layout finalized, production data generated
Parts:
- removed D11, D13, D9: LESD5D5.0CT1G, EasyBMS:SOD523_210, symbol EasyBMS-eagle-import:DIODE-SOD523
- removed D35, D36, D38: PESD5V0L1BA, Diode_SMD:D_SOD-323, symbol Diode:SD05_SOD323
- removed D37: LESD5D5.0CT1G, Diode_SMD:D_SOD-523, symbol Diode:ESD5Zxx
- removed U4, U6: RJ-064-1, RJ45 Connectors:CONN-SMD_RJ-064, symbol RJ45 Connectors:RJ-064-1
- added C60: 1nF/2000V, EasyBMS:C1206_334, symbol EasyBMS-eagle-import:C-EUC0805
- added D11, D13, D37, D9: LESD5D5.0CT1G_C5199850, EasyEDA2KiCAD:SOD-523_L1.2-W0.8-LS1.6-BI, symbol EasyEDA2KiCAD:LESD5D5.0CT1G_C5199850
- added D35: PESD1CAN,215, EasyEDA2KiCAD:SOT-23_L2.9-W1.3-P1.90-LS2.4-BR, symbol EasyEDA2KiCAD:PESD1CAN,215
- added H6: MOUNT-HOLE3.2, EasyBMS:3,2_237, symbol EasyBMS-eagle-import:MOUNT-HOLE3.2
- added L2: 10uH, Resistor_SMD:R_0805_2012Metric, symbol Device:L
- added R61: 1M, EasyBMS:R1206_334, symbol EasyBMS-eagle-import:R-EU_R1206
- added RJ1, RJ2: MJ88-B211-JRS3, EasyEDA2KiCAD:RJ45-SMD_HELING_MJ88-B211-JRS3, symbol EasyEDA2KiCAD:MJ88-B211-JRS3
- B1, BOOT0, H1, H2, H3, J2, JP1, RS485-AP1, RS485-BP1, RS485-GNDPWR1, RS485-VDD1, RST0, RX0, TERM0, TX0, U2, U7: now left out of the parts list
- C57, C58: LCSC (none) -> C107135
- IC1: footprint EasyBMS:SOIC127P600X170-9N -> EasyEDA2KiCAD:ESOP-8_L4.9-W3.9-P1.27-LS6.0-TL-EP
- IC6: LCSC (none) -> C6187
- LED2: footprint EasyBMS:XL-1615RGBC-WS2812B -> EasyEDA2KiCAD:LED-SMD_4P-L1.6-W1.5_XL-1615RGBC-WS2812B-1
- R1, R22, R92, R93: LCSC (none) -> C23185
- R24: LCSC (none) -> C25744
- U3: LCSC (none) -> C87626
Connections:
- net +12V: now also C2.1, LED2.3 (VDD), L2.2, RJ1.2; no longer LED2.VDD
- net +3V3: no longer C2.1, U7.2 (+Vin)
- net D+: now also D13.2
- net D-: now also D11.2
- net GND: now also LED2.1 (GND), D11.1, D13.1, D9.1; no longer LED2.VSS (GND)
- net GNDPWR: now also RJ1.3; no longer B1.0V
- net at C11.1, C18.1, J2.1 (Pin_1)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: now also D37.2
- net at C11.2, C18.2, CAN-GNDP1.2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: now also C60.1, D35.3, D37.1, R61.2
- net at CAN-GNDV1.1: now also RJ2.3
- net at CAN-HP1.1: now also RJ2.4
- net at CAN-LP1.1: now also RJ2.5
- net at CAN-GNDP1.1: now also RJ2.6
- net at CAN-HV1.1, RS485-AP1.2: now also RJ2.7
- net at CAN-LV1.1, RS485-BP1.2: now also RJ2.8
- net at D2.A, J1.A4_B9 (VBUS), J1.B4_A9 (VBUS): now also D9.2
- net at F2.1, R12.1, U5.6 (CANL): now also D35.2
- net at F1.1, TERM0.1, U5.7 (CANH): now also D35.1
- net at B1.A+, RS485-AP1.1: now also RJ1.4
- net at B1.B-, RS485-BP1.1: now also RJ1.5
- net at D15.2 (A), R21.2: now also LED2.2 (DI); no longer LED2.DIN (DI)
- new net: L2.1, U7.2 (+Vin)
- new net Earth: B1.0V, C60.2, R61.1, RJ1.10, RJ1.9, RJ2.10, RJ2.9
- no-connect marks 12 -> 15
Other:
- moved on the sheet: C2, CAN-HP1, CAN-HV1, CAN-LP1, CAN-LV1, F1, F2, J2

Commit message: new RGB LED and additional simple red LED
Parts:
- removed LED2: XL-1615RGBC-WS2812B, EasyEDA2KiCAD:LED-SMD_4P-L1.6-W1.5_XL-1615RGBC-WS2812B-1, symbol EasyBMS-eagle-import:XL-1615RGBC-WS2812B
- added D36: LED, LED_SMD:LED_0603_1608Metric, symbol Device:LED
- added R79: 1k, EasyBMS:R0402, symbol EasyBMS-eagle-import:R-EU_R0402
- added U4: XL-0807RGBC-WS2812B, EasyEDA2KiCAD:LED-SMD_4P-L2.0-W1.8_XL-0807RGBC-WS2812B, symbol EasyEDA2KiCAD:XL-0807RGBC-WS2812B
- B1: footprint RS485 Modul:RS-485-MODULE -> RS485Module:RS-485-MODULE
- C10, C11, C13, C15, C16, C17, C22, C42, C5, C56, C6, C61, C62, C66, C9: footprint EasyBMS:C0402_334 -> EasyBMS:C0402
- C12, C18, C64, C65, C7: footprint EasyBMS:C0805_334 -> EasyBMS:C0603
- C14, C21, C57, C58, C59: footprint EasyBMS:C0805_334 -> EasyBMS:C0805
- C24, C26: footprint EasyBMS:153CLV-0605_334 -> EasyBMS:153CLV-0605
- C27, C8: footprint EasyBMS:C0603_334 -> EasyBMS:C0603
- C60: footprint EasyBMS:C1206_334 -> EasyBMS:C0805
- CAN-GNDP1, CAN-GNDV1, CAN-HP1, CAN-HV1, CAN-LP1, CAN-LV1, IP-/GND1, RS485-AP1, RS485-BP1, RS485-GNDPWR1, RS485-VDD1, TERM0: footprint EasyBMS:SJ_252 -> EasyBMS:SJ
- D15: footprint EasyBMS:SOD3715X135_16378169 -> EasyBMS:SOD3715X135
- D2, D3: footprint EasyBMS:DO214AC_210 -> EasyBMS:DO214AC
- H1, H2, H3, H6: footprint EasyBMS:3,2_237 -> EasyBMS:3,2
- IC1: footprint EasyEDA2KiCAD:ESOP-8_L4.9-W3.9-P1.27-LS6.0-TL-EP -> EasyBMS:SOIC127P600X170-9N
- IC4, IC6: footprint EasyBMS:SOT223_111 -> EasyBMS:SOT223
- JP1: footprint EasyBMS:1X08_16378166 -> EasyBMS:1X08
- Q13: footprint Package_TO_SOT_SMD:SOT-223 -> Package_TO_SOT_SMD:SOT-223-3_TabPin2
- R1, R22, R90, R92, R93: footprint EasyBMS:R0603_334 -> EasyBMS:R0603
- R10, R11, R12, R13, R14, R2, R20, R21, R24, R5, R55, R6: footprint EasyBMS:R0402_334 -> EasyBMS:R0402
- R15, R16: footprint EasyBMS:R0603_334 -> EasyBMS:R0402
- R18, R19, R59, R61: footprint EasyBMS:R1206_334 -> EasyBMS:R1206
- RST0: footprint EasyBMS:B3F-10XX_377 -> EasyBMS:B3F-10XX
- RX0, TX0: footprint EasyBMS:B2,54_385 -> EasyBMS:B2,54
- U5: footprint Package_SO:SOIC-8_7.5x5.85mm_P1.27mm -> Package_SO:SOP-8_6.62x9.15mm_P2.54mm
Connections:
- net +12V: now also U4.4 (VDD)
- net GND: now also D36.1 (K), U4.2 (GND)
- net LED: now reaches U1.20 (IO15)
- net LED: now also R79.1
- net at D15.2 (A), R21.2: now also U4.3 (DIN)
- new net: D36.2 (A), R79.2
- no-connect marks 15 -> 14
Other:
- sheet Cell Pack 1: file call_pack_1.kicad_sch -> cell_pack_1.kicad_sch
- moved on the sheet: C17
