File: Dual-Version/cell_pack_1.kicad_sch (KiCad schematic)
At the start: 114 parts, among them IC2 LTC6811IG-1, Q14 CJ2301, Q15 CJ2301, Q16 CJ2301, Q18 CJ2301, Q20 CJ2301, Q22 CJ2301, Q24 CJ2301, Q26 CJ2301, Q28 CJ2301, Q30 CJ2301, Q32 CJ2301, Q34 CJ2301

Commit message: new RGB LED and additional simple red LED
Parts:
- C1, C19, C23, C25, C28, C29, C31, C33, C35, C37, C39, C4, C41, C43, C45, C47: footprint EasyBMS:C0402_334 -> EasyBMS:C0402
- C20: footprint EasyBMS:C0805_334 -> EasyBMS:C0805
- D1, D7: footprint EasyBMS:DO214AC_210 -> EasyBMS:DO214AC
- GND2: footprint EasyBMS:SJ_252 -> EasyBMS:SJ
- R100, R101, R104, R105, R112, R113, R120, R121, R128, R129, R136, R137, R144, R145, R152, R153, R160, R161, R168, R169, R176, R177, R82, R96: footprint EasyBMS:R1206_334 -> EasyBMS:R1206
- R102, R103, R106, R107, R114, R115, R122, R123, R130, R131, R138, R139, R146, R147, R154, R155, R162, R163, R170, R171, R178, R179, R57, R58, R60, R9, R97, R98: footprint EasyBMS:R0402_334 -> EasyBMS:R0402
- R17, R23, R3, R4, R7, R8: footprint EasyBMS:R0603_334 -> EasyBMS:R0603
