File: Dual-Version/cell_pack_2.kicad_sch (KiCad schematic)
At the start: 125 parts, among them IC5 LTC6811IG-1#PBF, J4 RJ45_Shielded, J5 RJ45_Shielded, Q1 CJ2301, Q10 CJ2301, Q11 CJ2301, Q12 CJ2301, Q13 NSV1C201MZ4, Q2 CJ2301, Q3 CJ2301, Q4 CJ2301, Q5 CJ2301, Q6 CJ2301, Q7 CJ2301, Q8 CJ2301, Q9 CJ2301

Commit message: schematic improvements, parts changed, layout progress
Parts:
- removed C12+POWER1: SJ, EasyBMS:SJ_252, symbol EasyBMS-eagle-import:SJ
- removed C56: 10nF, symbol Device:C
- removed C59: 100nF, EasyBMS:C0805_334, symbol EasyBMS-eagle-import:C-EUC0805
- removed J4, J5: RJ45_Shielded, symbol Connector:RJ45_Shielded
- removed Q13: NSV1C201MZ4, Package_TO_SOT_SMD:SOT-223, symbol Transistor_BJT:BCP56
- removed R79: 600R@100MHz, EasyBMS:R1206_334, symbol EasyBMS-eagle-import:R-EU_R1206
- removed R90: 100R, EasyBMS:R0603_334, symbol EasyBMS-eagle-import:R-EU_R0603
- removed R92, R93: 49R9, EasyBMS:R0603_334, symbol EasyBMS-eagle-import:R-EU_R0603
- removed R94: 100R, EasyBMS:R0402_334, symbol EasyBMS-eagle-import:R-EU_R0402
- IC5: value LTC6811IG-1#PBF -> LTC6811IG-1
- renumbered C1-/GND1 to GND1
Connections:
- net GND1: now also GND1.1
- net VREG: no longer IC5.40 (ISOMD)
- net VTEMP1: now also IC5.29 (GPIO3); no longer IC5.28 (GPIO2)
- net VTEMP2: now also IC5.28 (GPIO2); no longer IC5.29 (GPIO3)
- net DRIVE: now reaches IC5.38 (DRIVE)
- net SDI: now reaches IC5.43 (SDI_(NC))
- net SDO: now reaches IC5.44 (SDO_(NC))
- net CURRENT_SENSE renamed CURRENTSENSE
- net IMA renamed CSBIMA
- net IPA renamed SCKIPA
- new net ISOMD: IC5.40 (ISOMD)
- no-connect marks 3 -> 1
Other:
- moved on the sheet: C52, C53, C54, C55, IC5, R84, R85, R88, R89, R91

Commit message: schematic and layout finalized, production data generated
Parts:
- D17, D19, D21, D23, D25, D26, D27, D28, D29, D30, D31, D32, GND1, IC5, JP14, JP15, JP16, JP17, JP18, JP19, JP20, JP21, JP22, JP23, JP24: now left out of the parts list
- R89, R91: LCSC (none) -> C21190
Changed lines of the file:
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@@
 		(polyline
 			(pts
-				(xy 82.55 232.41) (xy 195.58 232.41) (xy 195.58 207.01) (xy 82.55 207.01)
+				(xy 82.55 64.77) (xy 195.58 64.77) (xy 195.58 39.37) (xy 82.55 39.37)
 			)
 			(stroke
@@
 		(polyline
 			(pts
-				(xy 82.55 316.23) (xy 195.58 316.23) (xy 195.58 290.83) (xy 82.55 290.83)
+				(xy 82.55 148.59) (xy 195.58 148.59) (xy 195.58 123.19) (xy 82.55 123.19)
 			)
 			(stroke
@@
 		(polyline
 			(pts
-				(xy 82.55 120.65) (xy 195.58 120.65) (xy 195.58 95.25) (xy 82.55 95.25)
+				(xy 82.55 344.17) (xy 195.58 344.17) (xy 195.58 318.77) (xy 82.55 318.77)
 			)
 			(stroke
@@
 		(polyline
 			(pts
-				(xy 82.55 260.35) (xy 195.58 260.35) (xy 195.58 234.95) (xy 82.55 234.95)
+				(xy 82.55 232.41) (xy 195.58 232.41) (xy 195.58 207.01) (xy 82.55 207.01)
 			)
 			(stroke
@@
 		(polyline
 			(pts
-				(xy 82.55 64.77) (xy 195.58 64.77) (xy 195.58 39.37) (xy 82.55 39.37)
+				(xy 82.55 316.23) (xy 195.58 316.23) (xy 195.58 290.83) (xy 82.55 290.83)
 			)
 			(stroke
@@
 		(polyline
 			(pts
-				(xy 389.89 397.51) (xy 16.51 400.05) (xy 15.24 398.78) (xy 15.24 20.32) (xy 16.51 19.05) (xy 421.64 19.05)
-				(xy 389.89 21.59)
+				(xy 389.89 397.51) (xy 16.51 400.05) (xy 15.24 398.78) (xy 15.24 20.32) (xy 16.51 19.05) (xy 389.89 19.05)
 			)
 			(stroke
@@
 		(polyline
 			(pts
-				(xy 82.55 344.17) (xy 195.58 344.17) (xy 195.58 318.77) (xy 82.55 318.77)
+				(xy 82.55 92.71) (xy 195.58 92.71) (xy 195.58 67.31) (xy 82.55 67.31)
 			)
 			(stroke
@@
 		(polyline
 			(pts
-				(xy 82.55 148.59) (xy 195.58 148.59) (xy 195.58 123.19) (xy 82.55 123.19)
+				(xy 82.55 176.53) (xy 195.58 176.53) (xy 195.58 151.13) (xy 82.55 151.13)
 			)
 			(stroke
@@
 		(polyline
 			(pts
-				(xy 82.55 92.71) (xy 195.58 92.71) (xy 195.58 67.31) (xy 82.55 67.31)
+				(xy 82.55 260.35) (xy 195.58 260.35) (xy 195.58 234.95) (xy 82.55 234.95)
 			)
 			(stroke
@@
 		(polyline
 			(pts
-				(xy 82.55 176.53) (xy 195.58 176.53) (xy 195.58 151.13) (xy 82.55 151.13)
+				(xy 82.55 204.47) (xy 195.58 204.47) (xy 195.58 179.07) (xy 82.55 179.07)
 			)
 			(stroke
@@
 		(polyline
 			(pts
-				(xy 82.55 204.47) (xy 195.58 204.47) (xy 195.58 179.07) (xy 82.55 179.07)
+				(xy 82.55 120.65) (xy 195.58 120.65) (xy 195.58 95.25) (xy 82.55 95.25)
 			)
 			(stroke
@@
 		(length 2.54)
 		(shape round)
-		(at 421.64 19.05 270)
+		(at 389.89 19.05 270)
 		(fields_autoplaced yes)
 		(effects
@@
 		)
 		(property "Netclass" ""
-			(at -49.53 -7.62 0)
+			(at -81.28 -7.62 0)
 			(effects
 				(font
@@
 		)
 		(property "Component Class" "BMS Channel 2"
-			(at 424.18 18.3515 90)
+			(at 392.43 18.3515 90)
 			(effects
 				(font
@@
 		(unit 1)
 		(exclude_from_sim no)
-		(in_bom yes)
+		(in_bom no)
 		(on_board yes)
 		(dnp no)
@@
 		(unit 1)
 		(exclude_from_sim no)
-		(in_bom yes)
+		(in_bom no)
 		(on_board yes)
 		(dnp no)
@@
 		(unit 1)
 		(exclude_from_sim no)
-		(in_bom yes)
+		(in_bom no)
 		(on_board yes)
 		(dnp no)
@@
 		(unit 1)
 		(exclude_from_sim no)
-		(in_bom yes)
+		(in_bom no)
 		(on_board yes)
 		(dnp no)
@@
 		(unit 1)
 		(exclude_from_sim no)
-		(in_bom yes)
+		(in_bom no)
 		(on_board yes)
 		(dnp no)
@@
 		(unit 1)
 		(exclude_from_sim no)
-		(in_bom yes)
+		(in_bom no)
 		(on_board yes)
 		(dnp no)
@@
 		(unit 1)
 		(exclude_from_sim no)
-		(in_bom yes)
+		(in_bom no)
 		(on_board yes)
 		(dnp no)
@@
 		(unit 1)
 		(exclude_from_sim no)
-		(in_bom yes)
+		(in_bom no)
 		(on_board yes)
 		(dnp no)
@@
 		(unit 1)
 		(exclude_from_sim no)
-		(in_bom yes)
+		(in_bom no)
 		(on_board yes)
 		(dnp no)
@@
 		(unit 1)
 		(exclude_from_sim no)
-		(in_bom yes)
+		(in_bom no)
 		(on_board yes)
 		(dnp no)
@@
 		(unit 1)
 		(exclude_from_sim no)
-		(in_bom yes)
+		(in_bom no)
 		(on_board yes)
 		(dnp no)
@@
 		(unit 1)
 		(exclude_from_sim no)
-		(in_bom yes)
+		(in_bom no)
 		(on_board yes)
 		(dnp no)
@@
 		(unit 1)
 		(exclude_from_sim no)
-		(in_bom yes)
+		(in_bom no)
 		(on_board yes)
 		(dnp no)
@@
 		(unit 1)
 		(exclude_from_sim no)
-		(in_bom yes)
+		(in_bom no)
 		(on_board yes)
 		(dnp no)
@@
 		(unit 1)
 		(exclude_from_sim no)
-		(in_bom yes)
+		(in_bom no)
 		(on_board yes)
 		(dnp no)
@@
 		(unit 1)
 		(exclude_from_sim no)
-		(in_bom yes)
+		(in_bom no)
 		(on_board yes)
 		(dnp no)
@@
 		(unit 1)
 		(exclude_from_sim no)
-		(in_bom yes)
+		(in_bom no)
 		(on_board yes)
 		(dnp no)
@@
 			)
 		)
-		(property "LCSC" ""
+		(property "LCSC" "C21190"
 			(at 477.52 205.74 0)
 			(effects
@@
 		(unit 1)
 		(exclude_from_sim no)
-		(in_bom yes)
+		(in_bom no)
 		(on_board yes)
 		(dnp no)
@@
 		(unit 1)
 		(exclude_from_sim no)
-		(in_bom yes)
+		(in_bom no)
 		(on_board yes)
 		(dnp no)
@@
 		(unit 1)
 		(exclude_from_sim no)
-		(in_bom yes)
+		(in_bom no)
 		(on_board yes)
 		(dnp no)
@@
 			)
 		)
-		(property "LCSC" ""
+		(property "LCSC" "C21190"
 			(at 491.49 205.74 0)
 			(effects
@@
 		(unit 1)
 		(exclude_from_sim no)
-		(in_bom yes)
+		(in_bom no)
 		(on_board yes)
 		(dnp no)
@@
 		(unit 1)
 		(exclude_from_sim no)
-		(in_bom yes)
+		(in_bom no)
 		(on_board yes)
 		(dnp no)
@@
 		(unit 1)
 		(exclude_from_sim no)
-		(in_bom yes)
+		(in_bom no)
 		(on_board yes)
 		(dnp no)
@@
 		(unit 1)
 		(exclude_from_sim no)
-		(in_bom yes)
+		(in_bom no)
 		(on_board yes)
 		(dnp no)
@@
 		(unit 1)
 		(exclude_from_sim no)
-		(in_bom yes)
+		(in_bom no)
 		(on_board yes)
 		(dnp no)

Commit message: new RGB LED and additional simple red LED
Parts:
- C3, C30, C32, C34, C36, C38, C40, C44, C46, C48, C49, C50, C51, C53, C54, C55: footprint EasyBMS:C0402_334 -> EasyBMS:C0402
- C52: footprint EasyBMS:C0805_334 -> EasyBMS:C0805
- D33, D34: footprint EasyBMS:DO214AC_210 -> EasyBMS:DO214AC
- GND1: footprint EasyBMS:SJ_252 -> EasyBMS:SJ
- R25, R26, R27, R28, R29, R30, R31, R32, R33, R34, R35, R36, R37, R38, R39, R40, R41, R42, R43, R44, R45, R46, R47, R48: footprint EasyBMS:R1206_334 -> EasyBMS:R1206
- R49, R50, R51, R52, R53, R54, R56, R62, R63, R64, R65, R66, R67, R68, R69, R70, R71, R72, R73, R74, R75, R76, R77, R78, R80, R84, R85, R88: footprint EasyBMS:R0402_334 -> EasyBMS:R0402
- R81, R83, R86, R87, R89, R91: footprint EasyBMS:R0603_334 -> EasyBMS:R0603
