File: RJ45 Adapter/RJ45 Adapter.kicad_pcb (KiCad board)
At the start: 2 copper layers, 30.7 x 44.4 mm, 13 parts

Commit message: schematic and layout finalized, production data generated
Parts:
- RJ1, RJ2: footprint RJ45 Connectors:RJ45-SMD_HELING_MJ88-B211-JRS3 -> EasyEDA2KiCAD:RJ45-SMD_HELING_MJ88-B211-JRS3
Changed lines of the file:
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@@
 		(sheetname "/")
 		(sheetfile "RJ45 Adapter.kicad_sch")
-		(attr through_hole)
+		(attr through_hole exclude_from_pos_files)
 		(fp_line
 			(start -1.33 3.87)
@@
 		(sheetname "/")
 		(sheetfile "RJ45 Adapter.kicad_sch")
-		(attr through_hole)
+		(attr through_hole exclude_from_pos_files)
 		(fp_line
 			(start 1.33 -1.33)
@@
 		(sheetname "/")
 		(sheetfile "RJ45 Adapter.kicad_sch")
-		(attr through_hole)
+		(attr through_hole exclude_from_pos_files)
 		(fp_line
 			(start -1.33 3.87)
@@
 		(sheetname "/")
 		(sheetfile "RJ45 Adapter.kicad_sch")
-		(attr through_hole)
+		(attr through_hole exclude_from_pos_files)
 		(fp_line
 			(start -1.33 3.87)
@@
 		(sheetname "/")
 		(sheetfile "RJ45 Adapter.kicad_sch")
-		(attr through_hole)
+		(attr through_hole exclude_from_pos_files)
 		(fp_line
 			(start -1.33 3.87)
@@
 		(sheetname "/")
 		(sheetfile "RJ45 Adapter.kicad_sch")
-		(attr through_hole)
+		(attr through_hole exclude_from_pos_files)
 		(fp_line
 			(start -1.33 3.87)
@@
 		(sheetname "/")
 		(sheetfile "RJ45 Adapter.kicad_sch")
-		(attr through_hole)
+		(attr through_hole exclude_from_pos_files)
 		(fp_line
 			(start 1.33 -1.33)
@@
 		(sheetname "/")
 		(sheetfile "RJ45 Adapter.kicad_sch")
-		(attr through_hole)
+		(attr through_hole exclude_from_pos_files)
 		(fp_line
 			(start -1.33 3.87)
@@
 		)
 	)
-	(footprint "RJ45 Connectors:RJ45-SMD_HELING_MJ88-B211-JRS3"
+	(footprint "EasyEDA2KiCAD:RJ45-SMD_HELING_MJ88-B211-JRS3"
 		(layer "F.Cu")
 		(at 76.825 44.815 -90)
 		(property "Reference" "RJ2"
-			(at 0 -11.46 90)
+			(at 0 -11.46 270)
 			(layer "F.SilkS")
 			(effects
@@
 		)
 		(property "Value" "MJ88-B211-JRS3"
-			(at 0 11.46 90)
+			(at 0 11.46 270)
 			(layer "F.Fab")
 			(effects
@@
 		)
 		(property "Datasheet" ""
-			(at 0 0 90)
+			(at 0 0 270)
 			(layer "F.Fab")
 			(hide yes)
@@
 		)
 		(property "Description" ""
-			(at 0 0 90)
+			(at 0 0 270)
 			(layer "F.Fab")
 			(hide yes)
@@
 		)
 		(fp_text user "${REFERENCE}"
-			(at 0 0 90)
+			(at 0 0 270)
 			(layer "F.Fab")
 			(effects
@@
 		)
 		(embedded_fonts no)
-		(model "${EASYEDA2KICAD}/easyeda2kicad.3dshapes/RJ45-SMD_HELING_MJ88-B211-JRS3.wrl"
+		(model "${KIPRJMOD}/../libraries/EasyEDA2KiCAD.3dshapes/RJ45-SMD_HELING_MJ88-B211-JRS3.wrl"
 			(offset
-				(xyz 0 -2.19 2.8)
+				(xyz 0 -2.19 11.8)
 			)
 			(scale
@@
 			)
 			(rotate
-				(xyz 0 0 0)
+				(xyz -0 -0 -0)
 			)
 		)
@@
 		(sheetname "/")
 		(sheetfile "RJ45 Adapter.kicad_sch")
-		(attr through_hole)
+		(attr through_hole exclude_from_pos_files)
 		(fp_line
 			(start 1.33 -1.33)
@@
 		(sheetname "/")
 		(sheetfile "RJ45 Adapter.kicad_sch")
-		(attr through_hole)
+		(attr through_hole exclude_from_pos_files)
 		(fp_line
 			(start -1.33 3.87)
@@
 		(sheetname "/")
 		(sheetfile "RJ45 Adapter.kicad_sch")
-		(attr through_hole)
+		(attr through_hole exclude_from_pos_files)
 		(fp_line
 			(start -1.33 3.87)
@@
 		)
 	)
-	(footprint "RJ45 Connectors:RJ45-SMD_HELING_MJ88-B211-JRS3"
+	(footprint "EasyEDA2KiCAD:RJ45-SMD_HELING_MJ88-B211-JRS3"
 		(layer "F.Cu")
 		(at 76.825 65.275 -90)
 		(property "Reference" "RJ1"
-			(at 0 -11.46 90)
+			(at 0 -11.46 270)
 			(layer "F.SilkS")
 			(effects
@@
 		)
 		(property "Value" "MJ88-B211-JRS3"
-			(at 0 11.46 90)
+			(at 0 11.46 270)
 			(layer "F.Fab")
 			(effects
@@
 		)
 		(property "Datasheet" ""
-			(at 0 0 90)
+			(at 0 0 270)
 			(layer "F.Fab")
 			(hide yes)
@@
 		)
 		(property "Description" ""
-			(at 0 0 90)
+			(at 0 0 270)
 			(layer "F.Fab")
 			(hide yes)
@@
 		)
 		(fp_text user "${REFERENCE}"
-			(at 0 0 90)
+			(at 0 0 270)
 			(layer "F.Fab")
 			(effects
@@
 		)
 		(embedded_fonts no)
-		(model "${EASYEDA2KICAD}/easyeda2kicad.3dshapes/RJ45-SMD_HELING_MJ88-B211-JRS3.wrl"
+		(model "${KIPRJMOD}/../libraries/EasyEDA2KiCAD.3dshapes/RJ45-SMD_HELING_MJ88-B211-JRS3.wrl"
 			(offset
-				(xyz 0 -2.19 2.8)
+				(xyz 0 -2.19 11.8)
 			)
 			(scale
@@
 			)
 			(rotate
-				(xyz 0 0 0)
+				(xyz -0 -0 -0)
 			)
 		)
