File: RJ45 Adapter/RJ45 Adapter.kicad_sch (KiCad schematic)
At the start: 13 parts

Commit message: schematic and layout finalized, production data generated
Parts:
- RJ1, RJ2: footprint RJ45 Connectors:RJ45-SMD_HELING_MJ88-B211-JRS3 -> EasyEDA2KiCAD:RJ45-SMD_HELING_MJ88-B211-JRS3; symbol RJ45 Connectors:MJ88-B211-JRS3 -> EasyEDA2KiCAD:MJ88-B211-JRS3
Changed lines of the file:
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@@
 	)
 	(symbol
-		(lib_id "RJ45 Connectors:MJ88-B211-JRS3")
+		(lib_id "EasyEDA2KiCAD:MJ88-B211-JRS3")
 		(at 234.95 114.3 180)
 		(unit 1)
@@
 		(fields_autoplaced yes)
 		(property "Reference" "RJ1"
-			(at 222.25 115.57 90)
-			(effects
-				(font
-					(size 1.27 1.27)
-				)
+			(at 246.38 114.2999 0)
+			(effects
+				(font
+					(size 1.27 1.27)
+				)
+				(justify right)
 			)
 		)
 		(property "Value" "MJ88-B211-JRS3"
-			(at 224.79 115.57 90)
-			(effects
-				(font
-					(size 1.27 1.27)
-				)
-			)
-		)
-		(property "Footprint" "RJ45 Connectors:RJ45-SMD_HELING_MJ88-B211-JRS3"
+			(at 246.38 116.8399 0)
+			(effects
+				(font
+					(size 1.27 1.27)
+				)
+				(justify right)
+			)
+		)
+		(property "Footprint" "EasyEDA2KiCAD:RJ45-SMD_HELING_MJ88-B211-JRS3"
 			(at 234.95 93.98 0)
 			(effects
@@
 	)
 	(symbol
-		(lib_id "RJ45 Connectors:MJ88-B211-JRS3")
+		(lib_id "EasyEDA2KiCAD:MJ88-B211-JRS3")
 		(at 57.15 115.57 180)
 		(unit 1)
@@
 		(fields_autoplaced yes)
 		(property "Reference" "RJ2"
-			(at 44.45 116.84 90)
-			(effects
-				(font
-					(size 1.27 1.27)
-				)
+			(at 68.58 115.5699 0)
+			(effects
+				(font
+					(size 1.27 1.27)
+				)
+				(justify right)
 			)
 		)
 		(property "Value" "MJ88-B211-JRS3"
-			(at 46.99 116.84 90)
-			(effects
-				(font
-					(size 1.27 1.27)
-				)
-			)
-		)
-		(property "Footprint" "RJ45 Connectors:RJ45-SMD_HELING_MJ88-B211-JRS3"
+			(at 68.58 118.1099 0)
+			(effects
+				(font
+					(size 1.27 1.27)
+				)
+				(justify right)
+			)
+		)
+		(property "Footprint" "EasyEDA2KiCAD:RJ45-SMD_HELING_MJ88-B211-JRS3"
 			(at 57.15 95.25 0)
 			(effects
